File: packages/addressable-leds/layouts/default/sk6805-ec20.kicad_pcb (KiCad board)
At the start: 2 copper layers, 2 parts

Commit message: WIP
Parts:
- C1: footprint atopile:C0402-b3ef17 -> SAMSUNG_CL05B104KO5NNNC:C0402
- U1: footprint lib:LED-SMD_4P-L2.0-W2.0-BR -> OPSCO_SK6805_EC20:LED-SMD_4P-L2.0-W2.0-BR
Connections:
- net DIN renamed package.footprint.pins[3].net-net
- net DOUT renamed package.footprint.pins[1].net-net
- U1 pad 1: VDD -> package.footprint.pins[0].net-net
- U1 pad 3: gnd -> package.footprint.pins[2].net-net

Commit message: update addressable leds
Parts:
- C1: footprint SAMSUNG_CL05B104KO5NNNC:C0402 -> Samsung_Electro_Mechanics_CL05B104KO5NNNC:C0402
Connections:
- net package.footprint.pins[1].net-net renamed DOUT
- net package.footprint.pins[3].net-net renamed DIN
- U1 pad 1: package.footprint.pins[0].net-net -> VDD
- U1 pad 3: package.footprint.pins[2].net-net -> gnd
Routing:
- net (no net): track 0.00 -> 5.55 mm, vias 0 -> 3
- net gnd: track 4.20 -> 0.00 mm, vias 2 -> 0
- net VDD: track 1.35 -> 0.00 mm, vias 1 -> 0
Changed lines of the file:
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@@
     )
     (net 0 "")
-    (net 1 "gnd")
-    (net 2 "package.footprint.pins[1].net-net")
-    (net 3 "package.footprint.pins[3].net-net")
-    (net 4 "VDD")
-    (net 5 "package.footprint.pins[0].net-net")
-    (net 6 "package.footprint.pins[2].net-net")
-    (footprint "SAMSUNG_CL05B104KO5NNNC:C0402"
+    (net 2 "DOUT")
+    (net 3 "DIN")
+    (net 7 "gnd")
+    (net 8 "VDD")
+    (footprint "Samsung_Electro_Mechanics_CL05B104KO5NNNC:C0402"
         (layer "F.Cu")
         (at 137.87 67.62 180)
@@
             )
         )
-        (property "__atopile_lib_fp_hash__" "899a684b-8724-fa64-4179-805a1b689684"
+        (property "__atopile_lib_fp_hash__" "c727fe38-bf01-b46b-3536-d9fd3e494ca3"
             (at 0 0 0)
             (layer "User.9")
@@
             )
         )
-        (property "checksum" "0254ae111d39f93a3986e7264696bf52c2f44f7516340732d4a1bfd3d039599c"
+        (property "checksum" "8df7e8fd450e964ff4be0fb3c3835c8921db5186cc940d09e4ccdc33aa93cf34"
             (at 0 0 0)
             (layer "User.9")
@@
             (size 0.79 0.54)
             (layers "F.Cu" "F.Paste" "F.Mask")
-            (net 1 "gnd")
+            (net 7 "gnd")
         )
         (pad "1" smd rect
@@
             (size 0.79 0.54)
             (layers "F.Cu" "F.Paste" "F.Mask")
-            (net 4 "VDD")
-        )
-        (model "${KIPRJMOD}/../../parts/SAMSUNG_CL05B104KO5NNNC/C0402_L1.0-W0.5-H0.5.step"
+            (net 8 "VDD")
+        )
+        (model "${KIPRJMOD}/../../parts/Samsung_Electro_Mechanics_CL05B104KO5NNNC/C0402_L1.0-W0.5-H0.5.step"
             (offset
                 (xyz 0 0 0)
@@
             (size 0.8 0.8)
             (layers "F.Cu" "F.Paste" "F.Mask")
-            (net 2 "package.footprint.pins[1].net-net")
+            (net 2 "DOUT")
         )
         (pad "1" smd rect
@@
             (size 0.8 0.8)
             (layers "F.Cu" "F.Paste" "F.Mask")
-            (net 5 "package.footprint.pins[0].net-net")
+            (net 8 "VDD")
         )
         (pad "4" smd rect
@@
             (size 0.8 0.8)
             (layers "F.Cu" "F.Paste" "F.Mask")
-            (net 3 "package.footprint.pins[3].net-net")
+            (net 3 "DIN")
         )
         (pad "3" smd rect
@@
             (size 0.8 0.8)
             (layers "F.Cu" "F.Paste" "F.Mask")
-            (net 6 "package.footprint.pins[2].net-net")
+            (net 7 "gnd")
         )
         (model "${KIPRJMOD}/../../parts/OPSCO_SK6805_EC20/LED-SMD_4P-L2.0-W2.0-BR.step"
@@
         (drill 0.3)
         (layers "F.Cu" "B.Cu")
-        (net 1)
+        (net 0)
     )
     (via
@@
         (drill 0.3)
         (layers "F.Cu" "B.Cu")
-        (net 1)
+        (net 0)
     )
     (via
@@
         (drill 0.3)
         (layers "F.Cu" "B.Cu")
-        (net 4)
+        (net 0)
     )
     (embedded_fonts no)
@@
         (end 136.57 67.59)
         (width 0.2)
-        (net 1)
+        (net 0)
         (layer "F.Cu")
     )
@@
         (end 136.6 67.62)
         (width 0.2)
-        (net 1)
+        (net 0)
         (layer "F.Cu")
     )
@@
         (end 137.11 64.98)
         (width 0.2)
-        (net 1)
+        (net 0)
         (layer "F.Cu")
     )
@@
         (end 137.12 64.97)
         (width 0.2)
-        (net 1)
+        (net 0)
         (layer "F.Cu")
     )
@@
         (end 136.38 64.98)
         (width 0.2)
-        (net 1)
+        (net 0)
         (layer "B.Cu")
     )
@@
         (end 136.57 65.17)
         (width 0.2)
-        (net 1)
+        (net 0)
         (layer "B.Cu")
     )
@@
         (end 138.42 66.27)
         (width 0.2)
-        (net 4)
+        (net 0)
         (layer "F.Cu")
     )
@@
         (end 138.42 67.01)
         (width 0.2)
-        (net 4)
-        (layer "F.Cu")
-    )
+        (net 0)
+        (layer "F.Cu")
+    )
