File: packages/ti-lv284x/layouts/test-1v8/test-1v8.kicad_pcb (KiCad board)
At the start: 2 copper layers, 0 parts

Commit message: Upgrade ti-lv284x to KiCAD 9.0
Parts:
- added C1: 470nF ±20% 16V X5R, atopile:C0402-b3ef17, F.Cu at (0.00, 0.00)
- added C2: 4.7µF ±10% 25V X5R, atopile:C0805-3b2e55, F.Cu at (0.00, -40.0)
- added C3: 10µF ±10% 25V X5R, atopile:C0805-3b2e55, F.Cu at (0.00, -50.0)
- added R1: 10kΩ ±1% 62.5mW, atopile:R0402-56259e, F.Cu at (10.0, 0.00)
- added R2: 13kΩ ±1% 62.5mW, atopile:R0402-56259e, F.Cu at (10.0, -10.0)
- added U1: , lib:SOD-323_L1.8-W1.3-LS2.5-RD, F.Cu at (0.00, -30.0)
- added U2: , lib:SOT-23-6_L2.9-W1.6-P0.95-LS2.8-BR, F.Cu at (0.00, -10.0)
- added U3: 10µH ±20%, lib:IND-SMD_L4.0-W4.0, F.Cu at (0.00, -20.0)

Commit message: update LV2842 to build frozen
Parts:
- R1: value 10kΩ ±1% 62.5mW -> 8.06kΩ ±1% 62.5mW
- R2: value 13kΩ ±1% 62.5mW -> 10kΩ ±1% 62.5mW
Connections:
- C2 pad 2: gnd -> gnd-1
- C3 pad 2: gnd-1 -> gnd
- R1 pad 2: gnd-1 -> gnd
- U1 pad 2: gnd-1 -> gnd
- U2 pad 2: gnd -> gnd-1
Changed lines of the file:
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@@
     (net 3 "hv-1")
     (net 4 "FB")
-    (net 5 "gnd-1")
+    (net 5 "gnd")
     (net 6 "hv")
-    (net 7 "gnd")
+    (net 7 "gnd-1")
     (footprint "atopile:C0402-b3ef17"
         (layer "F.Cu")
@@
             (size 1.1 0.6)
             (layers "F.Cu" "F.Paste" "F.Mask")
-            (net 7 "gnd")
+            (net 7 "gnd-1")
         )
         (pad "1" smd rect
@@
             (size 1 0.75)
             (layers "F.Cu" "F.Paste" "F.Mask")
-            (net 5 "gnd-1")
+            (net 5 "gnd")
         )
         (pad "1" smd rect
@@
             (size 1.41 1.35)
             (layers "F.Cu" "F.Paste" "F.Mask")
-            (net 7 "gnd")
+            (net 7 "gnd-1")
         )
         (pad "1" smd rect
@@
             (size 1.41 1.35)
             (layers "F.Cu" "F.Paste" "F.Mask")
-            (net 5 "gnd-1")
+            (net 5 "gnd")
         )
         (pad "1" smd rect
@@
             )
         )
-        (property "Value" "10kΩ ±1% 62.5mW"
+        (property "Value" "8.06kΩ ±1% 62.5mW"
             (at 0 4 0)
             (layer "F.Fab")
@@
             )
         )
-        (property "LCSC" "C25744"
-            (at 0 0 0)
-            (layer "User.9")
-            (hide yes)
-            (effects
-                (font
-                    (size 0.125 0.125)
-                    (thickness 0.01875)
-                )
-            )
-        )
-        (property "Partnumber" "0402WGF1002TCE"
-            (at 0 0 0)
-            (layer "User.9")
-            (hide yes)
-            (effects
-                (font
-                    (size 0.125 0.125)
-                    (thickness 0.01875)
-                )
-            )
-        )
-        (property "Manufacturer" "UNI-ROYAL(Uniroyal Elec)"
-            (at 0 0 0)
-            (layer "User.9")
-            (hide yes)
-            (effects
-                (font
-                    (size 0.125 0.125)
-                    (thickness 0.01875)
-                )
-            )
-        )
-        (property "JLCPCB description" "62.5mW Thick Film Resistors 50V ±100ppm/℃ ±1% 10kΩ 0402 Chip Resistor - Surface Mount ROHS"
+        (property "LCSC" "C276278"
+            (at 0 0 0)
+            (layer "User.9")
+            (hide yes)
+            (effects
+                (font
+                    (size 0.125 0.125)
+                    (thickness 0.01875)
+                )
+            )
+        )
+        (property "Partnumber" "RC0402FR-078K06L"
+            (at 0 0 0)
+            (layer "User.9")
+            (hide yes)
+            (effects
+                (font
+                    (size 0.125 0.125)
+                    (thickness 0.01875)
+                )
+            )
+        )
+        (property "Manufacturer" "YAGEO"
+            (at 0 0 0)
+            (layer "User.9")
+            (hide yes)
+            (effects
+                (font
+                    (size 0.125 0.125)
+                    (thickness 0.01875)
+                )
+            )
+        )
+        (property "JLCPCB description" "62.5mW Thick Film Resistors 50V ±100ppm/℃ ±1% 8.06kΩ 0402  Chip Resistor - Surface Mount ROHS"
             (at 0 0 0)
             (layer "User.9")
@@
             )
         )
-        (property "PARAM_resistance" "{\"type\": \"Quantity_Interval_Disjoint\", \"data\": {\"intervals\": {\"type\": \"Numeric_Interval_Disjoint\", \"data\": {\"intervals\": [{\"type\": \"Numeric_Interval\", \"data\": {\"min\": 9900.000002235174, \"max\": 10099.999997764826}}]}}, \"unit\": \"ohm\"}}"
+        (property "PARAM_resistance" "{\"type\": \"Quantity_Interval_Disjoint\", \"data\": {\"intervals\": {\"type\": \"Numeric_Interval_Disjoint\", \"data\": {\"intervals\": [{\"type\": \"Numeric_Interval\", \"data\": {\"min\": 7979.400001801551, \"max\": 8140.5999981984505}}]}}, \"unit\": \"ohm\"}}"
             (at 0 0 0)
             (layer "User.9")
@@
             (size 0.57 0.54)
             (layers "F.Cu" "F.Paste" "F.Mask")
-            (net 5 "gnd-1")
+            (net 5 "gnd")
         )
         (pad "1" smd rect
@@
             )
         )
-        (property "Value" "13kΩ ±1% 62.5mW"
+        (property "Value" "10kΩ ±1% 62.5mW"
             (at 0 4 0)
             (layer "F.Fab")
@@
             )
         )
-        (property "LCSC" "C138057"
-            (at 0 0 0)
-            (layer "User.9")
-            (hide yes)
-            (effects
-                (font
-                    (size 0.125 0.125)
-                    (thickness 0.01875)
-                )
-            )
-        )
-        (property "Partnumber" "RC0402FR-0713KL"
-            (at 0 0 0)
-            (layer "User.9")
-            (hide yes)
-            (effects
-                (font
-                    (size 0.125 0.125)
-                    (thickness 0.01875)
-                )
-            )
-        )
-        (property "Manufacturer" "YAGEO"
-            (at 0 0 0)
-            (layer "User.9")
-            (hide yes)
-            (effects
-                (font
-                    (size 0.125 0.125)
-                    (thickness 0.01875)
-                )
-            )
-        )
-        (property "JLCPCB description" "62.5mW Thick Film Resistors 50V ±100ppm/℃ ±1% 13kΩ 0402 Chip Resistor - Surface Mount ROHS"
+        (property "LCSC" "C25744"
+            (at 0 0 0)
+            (layer "User.9")
+            (hide yes)
+            (effects
+                (font
+                    (size 0.125 0.125)
+                    (thickness 0.01875)
+                )
+            )
+        )
+        (property "Partnumber" "0402WGF1002TCE"
+            (at 0 0 0)
+            (layer "User.9")
+            (hide yes)
+            (effects
+                (font
+                    (size 0.125 0.125)
+                    (thickness 0.01875)
+                )
+            )
+        )
+        (property "Manufacturer" "UNI-ROYAL(Uniroyal Elec)"
+            (at 0 0 0)
+            (layer "User.9")
+            (hide yes)
+            (effects
+                (font
+                    (size 0.125 0.125)
+                    (thickness 0.01875)
+                )
+            )
+        )
+        (property "JLCPCB description" "62.5mW Thick Film Resistors 50V ±100ppm/℃ ±1% 10kΩ 0402 Chip Resistor - Surface Mount ROHS"
             (at 0 0 0)
             (layer "User.9")
@@
             )
         )
-        (property "PARAM_resistance" "{\"type\": \"Quantity_Interval_Disjoint\", \"data\": {\"intervals\": {\"type\": \"Numeric_Interval_Disjoint\", \"data\": {\"intervals\": [{\"type\": \"Numeric_Interval\", \"data\": {\"min\": 12870.000002905726, \"max\": 13129.999997094274}}]}}, \"unit\": \"ohm\"}}"
-            (at 0 0 0)
-            (layer "User.9")
+        (property "PARAM_resistance" "{\"type\": \"Quantity_Interval_Disjoint\", \"data\": {\"intervals\": {\"type\": \"Numeric_Interval_Disjoint\", \"data\": {\"intervals\": [{\"type\": \"Numeric_Interval\", \"data\": {\"min\": 9900.000002235174, \"max\": 10099.999997764826}}]}}, \"unit\": \"ohm\"}}"
+            (at 0 0 0)
+            (layer "User.9")

Commit message: WIP
Parts:
- removed U1: , lib:SOD-323_L1.8-W1.3-LS2.5-RD
- C1: footprint atopile:C0402-b3ef17 -> CCTC_TCC0402X5R474M160AT:C0402
- C2: footprint atopile:C0805-3b2e55 -> SAMSUNG_CL21A475KAQNNNE:C0805
- C3: footprint atopile:C0805-3b2e55 -> SAMSUNG_CL21A106KAYNNNE:C0805
- R1: value 8.06kΩ ±1% 62.5mW -> 10kΩ ±1% 62.5mW; footprint atopile:R0402-56259e -> UNI_ROYAL_0402WGF1002TCE:R0402
- R2: value 10kΩ ±1% 62.5mW -> 13kΩ ±1% 62.5mW; footprint atopile:R0402-56259e -> UNI_ROYAL_0402WGF1302TCE:R0402
- U2: footprint lib:SOT-23-6_L2.9-W1.6-P0.95-LS2.8-BR -> TI_LV2842XLVDDCR:SOT-23-6_L2.9-W1.6-P0.95-LS2.8-BR
- U3: footprint lib:IND-SMD_L4.0-W4.0 -> Sunlord_SWPA4030S100MT:IND-SMD_L4.0-W4.0
Connections:
- net gnd renamed regulator-gnd
- C1 pad 2: SW -> cathode
- C2 pad 1: hv-1 -> regulator.ic.footprint.pins[3].net-net
- C2 pad 2: gnd-1 -> regulator-gnd-1
- U2 pad 1: CB -> regulator.ic.footprint.pins[0].net-net
- U2 pad 2: gnd-1 -> regulator.ic.footprint.pins[1].net-net
- U2 pad 3: FB -> regulator.ic.footprint.pins[2].net-net
- U2 pad 4: hv-1 -> regulator.ic.footprint.pins[3].net-net
- U2 pad 5: hv-1 -> regulator.ic.footprint.pins[4].net-net
- U2 pad 6: SW -> regulator.ic.footprint.pins[5].net-net
- U3 pad 1: SW -> regulator.inductor.footprint.pins[0].net-net
- U3 pad 2: hv -> regulator.inductor.footprint.pins[1].net-net

Commit message: rebuild
Parts:
- R1: value 10kΩ ±1% 62.5mW -> 8.06kΩ ±1% 62.5mW; footprint UNI_ROYAL_0402WGF1002TCE:R0402 -> YAGEO_RC0402FR_078K06L:R0402
- R2: value 13kΩ ±1% 62.5mW -> 10kΩ ±1% 62.5mW; footprint UNI_ROYAL_0402WGF1302TCE:R0402 -> UNI_ROYAL_0402WGF1002TCE:R0402
- U3: value 10µH ±20% -> (none)
Connections:
- net cathode renamed K
- C2 pad 1: regulator.ic.footprint.pins[3].net-net -> nSHDN
- C2 pad 2: regulator-gnd-1 -> regulator-gnd
- C3 pad 2: regulator-gnd -> regulator-gnd-1
- R1 pad 2: regulator-gnd -> regulator-gnd-1

Commit message: add build_all.py
Parts:
- R1: value 8.06kΩ ±1% 62.5mW -> 10kΩ ±1% 62.5mW; footprint YAGEO_RC0402FR_078K06L:R0402 -> UNI_ROYAL_0402WGF1002TCE:R0402
- R2: value 10kΩ ±1% 62.5mW -> 13kΩ ±1% 62.5mW; footprint UNI_ROYAL_0402WGF1002TCE:R0402 -> UNI_ROYAL_0402WGF1302TCE:R0402
Connections:
- net K renamed cathode
- C2 pad 2: regulator-gnd -> regulator-gnd-1
- C3 pad 2: regulator-gnd-1 -> regulator-gnd
- R1 pad 2: regulator-gnd-1 -> regulator-gnd
Changed lines of the file:
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@@
     )
     (net 0 "")
-    (net 1 "K")
+    (net 1 "cathode")
     (net 2 "CB")
     (net 3 "nSHDN")
     (net 4 "FB")
-    (net 5 "regulator-gnd-1")
+    (net 5 "regulator-gnd")
     (net 6 "hv")
-    (net 7 "regulator-gnd")
+    (net 7 "regulator-gnd-1")
     (net 8 "regulator.ic.footprint.pins[4].net-net")
     (net 9 "regulator.ic.footprint.pins[0].net-net")
@@
             (size 0.79 0.54)
             (layers "F.Cu" "F.Paste" "F.Mask")
-            (net 1 "K")
+            (net 1 "cathode")
         )
         (pad "1" smd rect
@@
             (size 1.41 1.35)
             (layers "F.Cu" "F.Paste" "F.Mask")
-            (net 7 "regulator-gnd")
+            (net 7 "regulator-gnd-1")
         )
         (pad "1" smd rect
@@
             (size 1.41 1.35)
             (layers "F.Cu" "F.Paste" "F.Mask")
-            (net 5 "regulator-gnd-1")
+            (net 5 "regulator-gnd")
         )
         (pad "1" smd rect
@@
         )
     )
-    (footprint "YAGEO_RC0402FR_078K06L:R0402"
+    (footprint "UNI_ROYAL_0402WGF1002TCE:R0402"
         (layer "F.Cu")
         (at 10 0 0)
@@
             )
         )
-        (property "Value" "8.06kΩ ±1% 62.5mW"
+        (property "Value" "10kΩ ±1% 62.5mW"
             (at 0 4 0)
             (layer "F.Fab")
@@
             )
         )
-        (property "__atopile_lib_fp_hash__" "b930602a-fafc-7ce7-61f4-9a92910f5691"
-            (at 0 0 0)
-            (layer "User.9")
-            (hide yes)
-            (effects
-                (font
-                    (size 0.125 0.125)
-                    (thickness 0.01875)
-                )
-            )
-        )
-        (property "LCSC" "C276278"
-            (at 0 0 0)
-            (layer "User.9")
-            (hide yes)
-            (effects
-                (font
-                    (size 0.125 0.125)
-                    (thickness 0.01875)
-                )
-            )
-        )
-        (property "Partnumber" "RC0402FR-078K06L"
-            (at 0 0 0)
-            (layer "User.9")
-            (hide yes)
-            (effects
-                (font
-                    (size 0.125 0.125)
-                    (thickness 0.01875)
-                )
-            )
-        )
-        (property "Manufacturer" "YAGEO"
+        (property "__atopile_lib_fp_hash__" "52234549-8985-85d4-dd79-0d66742cf16c"
+            (at 0 0 0)
+            (layer "User.9")
+            (hide yes)
+            (effects
+                (font
+                    (size 0.125 0.125)
+                    (thickness 0.01875)
+                )
+            )
+        )
+        (property "LCSC" "C25744"
+            (at 0 0 0)
+            (layer "User.9")
+            (hide yes)
+            (effects
+                (font
+                    (size 0.125 0.125)
+                    (thickness 0.01875)
+                )
+            )
+        )
+        (property "Partnumber" "0402WGF1002TCE"
+            (at 0 0 0)
+            (layer "User.9")
+            (hide yes)
+            (effects
+                (font
+                    (size 0.125 0.125)
+                    (thickness 0.01875)
+                )
+            )
+        )
+        (property "Manufacturer" "UNI-ROYAL(Uniroyal Elec)"
             (at 0 0 0)
             (layer "User.9")
@@
             )
         )
-        (property "PARAM_resistance" "{\"type\": \"Quantity_Interval_Disjoint\", \"data\": {\"intervals\": {\"type\": \"Numeric_Interval_Disjoint\", \"data\": {\"intervals\": [{\"type\": \"Numeric_Interval\", \"data\": {\"min\": 7979.400001801551, \"max\": 8140.5999981984505}}]}}, \"unit\": \"ohm\"}}"
+        (property "PARAM_resistance" "{\"type\": \"Quantity_Interval_Disjoint\", \"data\": {\"intervals\": {\"type\": \"Numeric_Interval_Disjoint\", \"data\": {\"intervals\": [{\"type\": \"Numeric_Interval\", \"data\": {\"min\": 9900.000002235174, \"max\": 10099.999997764826}}]}}, \"unit\": \"ohm\"}}"
             (at 0 0 0)
             (layer "User.9")
@@
             )
         )
-        (property "checksum" "facd2cceb9913cd43e2197006ffbe0aca6d15e0dfb3236c95eaf1534f75eca7c"
+        (property "checksum" "259c8f2b3c4ed145b90b418853b1dc377fc6c3fd12e0e8205ed5f17f665dfda4"
             (at 0 0 0)
             (layer "User.9")
@@
             )
         )
-        (property "Datasheet" "https://wmsc.lcsc.com/wmsc/upload/file/pdf/v2/lcsc/2304140030_YAGEO-RC0402FR-078K06L_C276278.pdf"
+        (property "Datasheet" "https://www.lcsc.com/datasheet/lcsc_datasheet_2411221126_UNI-ROYAL-Uniroyal-Elec-0402WGF1002TCE_C25744.pdf"
             (at 0 0 0)
             (layer "User.9")
@@
             (size 0.57 0.54)
             (layers "F.Cu" "F.Paste" "F.Mask")
-            (net 5 "regulator-gnd-1")
+            (net 5 "regulator-gnd")
         )
         (pad "1" smd rect
@@
             (net 4 "FB")
         )
-        (model "${KIPRJMOD}/../../build/cache/parts/easyeda/C276278/R0402_L1.0-W0.5-H0.4.step"
+        (model "${KIPRJMOD}/../../parts/UNI_ROYAL_0402WGF1002TCE/R0402_L1.0-W0.5-H0.4.step"
             (offset
                 (xyz 0 0 0)
@@
         )
     )
-    (footprint "UNI_ROYAL_0402WGF1002TCE:R0402"
+    (footprint "UNI_ROYAL_0402WGF1302TCE:R0402"
         (layer "F.Cu")
         (at 10 -10 0)
@@
             )
         )
-        (property "Value" "10kΩ ±1% 62.5mW"
+        (property "Value" "13kΩ ±1% 62.5mW"
             (at 0 4 0)
             (layer "F.Fab")
@@
             )
         )
-        (property "__atopile_lib_fp_hash__" "52234549-8985-85d4-dd79-0d66742cf16c"
-            (at 0 0 0)
-            (layer "User.9")
-            (hide yes)
-            (effects
-                (font
-                    (size 0.125 0.125)
-                    (thickness 0.01875)
-                )
-            )
-        )
-        (property "LCSC" "C25744"
-            (at 0 0 0)
-            (layer "User.9")
-            (hide yes)
-            (effects
-                (font
-                    (size 0.125 0.125)
-                    (thickness 0.01875)
-                )
-            )
-        )
-        (property "Partnumber" "0402WGF1002TCE"
+        (property "__atopile_lib_fp_hash__" "d23ef272-7714-8627-8e8c-b329de092641"
+            (at 0 0 0)
+            (layer "User.9")
+            (hide yes)
+            (effects
+                (font
+                    (size 0.125 0.125)
+                    (thickness 0.01875)
+                )
+            )
+        )
+        (property "LCSC" "C25754"
+            (at 0 0 0)
+            (layer "User.9")
+            (hide yes)
+            (effects
+                (font
+                    (size 0.125 0.125)
+                    (thickness 0.01875)
+                )
+            )
+        )
+        (property "Partnumber" "0402WGF1302TCE"
             (at 0 0 0)
             (layer "User.9")
@@
             )
         )
-        (property "PARAM_resistance" "{\"type\": \"Quantity_Interval_Disjoint\", \"data\": {\"intervals\": {\"type\": \"Numeric_Interval_Disjoint\", \"data\": {\"intervals\": [{\"type\": \"Numeric_Interval\", \"data\": {\"min\": 9900.000002235174, \"max\": 10099.999997764826}}]}}, \"unit\": \"ohm\"}}"
+        (property "PARAM_resistance" "{\"type\": \"Quantity_Interval_Disjoint\", \"data\": {\"intervals\": {\"type\": \"Numeric_Interval_Disjoint\", \"data\": {\"intervals\": [{\"type\": \"Numeric_Interval\", \"data\": {\"min\": 12870.000002905726, \"max\": 13129.999997094274}}]}}, \"unit\": \"ohm\"}}"
             (at 0 0 0)
             (layer "User.9")
@@
             )
         )
-        (property "checksum" "259c8f2b3c4ed145b90b418853b1dc377fc6c3fd12e0e8205ed5f17f665dfda4"
+        (property "checksum" "690c8ab5cf4d4b0d312e5a83f8315472834ca622651f25dfa304c2ccaaa63efe"
             (at 0 0 0)
             (layer "User.9")
@@
             )
         )
-        (property "Datasheet" "https://www.lcsc.com/datasheet/lcsc_datasheet_2411221126_UNI-ROYAL-Uniroyal-Elec-0402WGF1002TCE_C25744.pdf"
+        (property "Datasheet" "https://www.lcsc.com/datasheet/lcsc_datasheet_2206010100_UNI-ROYAL-Uniroyal-Elec-0402WGF1302TCE_C25754.pdf"
             (at 0 0 0)
             (layer "User.9")
@@
             (net 6 "hv")
         )
-        (model "${KIPRJMOD}/../../parts/UNI_ROYAL_0402WGF1002TCE/R0402_L1.0-W0.5-H0.4.step"
+        (model "${KIPRJMOD}/../../parts/UNI_ROYAL_0402WGF1302TCE/R0402_L1.0-W0.5-H0.4.step"
             (offset
                 (xyz 0 0 0)

Commit message: update ti-lv28 layout
Parts:
- added D1: , Hottech_1N5819WS:SOD-323_L1.8-W1.3-LS2.5-RD, F.Cu at (0.00, 0.00)
- C2: footprint SAMSUNG_CL21A475KAQNNNE:C0805 -> Samsung_Electro_Mechanics_CL21A475KAQNNNE:C0805
- C3: footprint SAMSUNG_CL21A106KAYNNNE:C0805 -> Samsung_Electro_Mechanics_CL21A106KAYNNNE:C0805
Connections:
- net regulator.inductor.footprint.pins[0].net-net renamed regulator.inductor-net-1
- net regulator.inductor.footprint.pins[1].net-net renamed regulator.inductor-net
- U2 pad 1: regulator.ic.footprint.pins[0].net-net -> CB
- U2 pad 2: regulator.ic.footprint.pins[1].net-net -> regulator-gnd-1
- U2 pad 3: regulator.ic.footprint.pins[2].net-net -> FB
- U2 pad 4: regulator.ic.footprint.pins[3].net-net -> nSHDN
- U2 pad 5: regulator.ic.footprint.pins[4].net-net -> nSHDN
- U2 pad 6: regulator.ic.footprint.pins[5].net-net -> cathode
