File: packages/ti-lv284x/layouts/test-3v3/test-3v3.kicad_pcb (KiCad board)
At the start: 2 copper layers, 0 parts

Commit message: Upgrade ti-lv284x to KiCAD 9.0
Parts:
- added C1: 470nF ±20% 16V X5R, atopile:C0402-b3ef17, F.Cu at (0.00, 0.00)
- added C2: 4.7µF ±10% 25V X5R, atopile:C0805-3b2e55, F.Cu at (0.00, -40.0)
- added C3: 10µF ±10% 25V X5R, atopile:C0805-3b2e55, F.Cu at (0.00, -50.0)
- added R1: 30kΩ ±1% 62.5mW, atopile:R0402-56259e, F.Cu at (10.0, 0.00)
- added R2: 100kΩ ±1% 62.5mW, atopile:R0402-56259e, F.Cu at (10.0, -10.0)
- added U1: , lib:SOD-323_L1.8-W1.3-LS2.5-RD, F.Cu at (0.00, -10.0)
- added U2: , lib:SOT-23-6_L2.9-W1.6-P0.95-LS2.8-BR, F.Cu at (0.00, -20.0)
- added U3: 10µH ±20%, lib:IND-SMD_L4.0-W4.0, F.Cu at (0.00, -30.0)

Commit message: update LV2842 to build frozen
Connections:
- net SW renamed cathode
- C2 pad 1: hv -> hv-1
- C3 pad 1: hv-1 -> hv
- R2 pad 1: hv-1 -> hv
- U2 pad 4: hv -> hv-1
- U2 pad 5: hv -> hv-1
- U3 pad 2: hv-1 -> hv
Changed lines of the file:
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@@
     (net 1 "CB")
     (net 2 "FB")
-    (net 3 "hv")
-    (net 4 "hv-1")
+    (net 3 "hv-1")
+    (net 4 "hv")
     (net 5 "gnd")
-    (net 6 "SW")
+    (net 6 "cathode")
     (net 7 "gnd-1")
     (footprint "atopile:C0402-b3ef17"
@@
             (size 0.79 0.54)
             (layers "F.Cu" "F.Paste" "F.Mask")
-            (net 6 "SW")
+            (net 6 "cathode")
         )
         (pad "1" smd rect
@@
             (size 1 0.75)
             (layers "F.Cu" "F.Paste" "F.Mask")
-            (net 6 "SW")
+            (net 6 "cathode")
         )
         (model "${KIPRJMOD}/../../../build/footprints/footprints.3dshapes/SOD-323_L1.7-W1.3-H1.1-LS2.5.step"
@@
             (size 1.1 0.6)
             (layers "F.Cu" "F.Paste" "F.Mask")
-            (net 6 "SW")
+            (net 6 "cathode")
         )
         (pad "5" smd rect
@@
             (size 1.1 0.6)
             (layers "F.Cu" "F.Paste" "F.Mask")
-            (net 3 "hv")
+            (net 3 "hv-1")
         )
         (pad "4" smd rect
@@
             (size 1.1 0.6)
             (layers "F.Cu" "F.Paste" "F.Mask")
-            (net 3 "hv")
+            (net 3 "hv-1")
         )
         (model "${KIPRJMOD}/../../../build/footprints/footprints.3dshapes/SOT-23-6_L2.9-W1.6-H1.5-LS2.8-P0.95.step"
@@
             (size 1.6 3.5)
             (layers "F.Cu" "F.Paste" "F.Mask")
-            (net 4 "hv-1")
+            (net 4 "hv")
         )
         (pad "1" smd rect
@@
             (size 1.6 3.5)
             (layers "F.Cu" "F.Paste" "F.Mask")
-            (net 6 "SW")
+            (net 6 "cathode")
         )
         (model "${KIPRJMOD}/../../../build/footprints/footprints.3dshapes/IND-SMD_L4.0-W4.0-H1.9.step"
@@
             (size 1.41 1.35)
             (layers "F.Cu" "F.Paste" "F.Mask")
-            (net 3 "hv")
+            (net 3 "hv-1")
         )
     )
@@
             (size 1.41 1.35)
             (layers "F.Cu" "F.Paste" "F.Mask")
-            (net 4 "hv-1")
+            (net 4 "hv")
         )
     )
@@
             (size 0.57 0.54)
             (layers "F.Cu" "F.Paste" "F.Mask")
-            (net 4 "hv-1")
+            (net 4 "hv")
         )
     )

Commit message: WIP
Parts:
- removed U1: , lib:SOD-323_L1.8-W1.3-LS2.5-RD
- C1: footprint atopile:C0402-b3ef17 -> CCTC_TCC0402X5R474M160AT:C0402
- C2: footprint atopile:C0805-3b2e55 -> SAMSUNG_CL21A475KAQNNNE:C0805
- C3: footprint atopile:C0805-3b2e55 -> SAMSUNG_CL21A106KAYNNNE:C0805
- R1: value 30kΩ ±1% 62.5mW -> 10kΩ ±1% 62.5mW; footprint atopile:R0402-56259e -> UNI_ROYAL_0402WGF1002TCE:R0402
- R2: value 100kΩ ±1% 62.5mW -> 33kΩ ±1% 62.5mW; footprint atopile:R0402-56259e -> UNI_ROYAL_0402WGF3302TCE:R0402
- U2: footprint lib:SOT-23-6_L2.9-W1.6-P0.95-LS2.8-BR -> TI_LV2842XLVDDCR:SOT-23-6_L2.9-W1.6-P0.95-LS2.8-BR
- U3: footprint lib:IND-SMD_L4.0-W4.0 -> Sunlord_SWPA4030S100MT:IND-SMD_L4.0-W4.0
Connections:
- net gnd renamed regulator-gnd
- C1 pad 2: cathode -> SW
- C2 pad 1: hv-1 -> VIN
- C2 pad 2: gnd-1 -> regulator-gnd-1
- U2 pad 1: CB -> regulator.ic.footprint.pins[0].net-net
- U2 pad 2: gnd-1 -> regulator.ic.footprint.pins[1].net-net
- U2 pad 3: FB -> regulator.ic.footprint.pins[2].net-net
- U2 pad 4: hv-1 -> regulator.ic.footprint.pins[3].net-net
- U2 pad 5: hv-1 -> regulator.ic.footprint.pins[4].net-net
- U2 pad 6: cathode -> regulator.ic.footprint.pins[5].net-net
- U3 pad 1: cathode -> regulator.inductor.footprint.pins[0].net-net
- U3 pad 2: hv -> regulator.inductor.footprint.pins[1].net-net

Commit message: rebuild
Parts:
- R1: value 10kΩ ±1% 62.5mW -> 30kΩ ±1% 62.5mW; footprint UNI_ROYAL_0402WGF1002TCE:R0402 -> UNI_ROYAL_0402WGF3002TCE:R0402
- R2: value 33kΩ ±1% 62.5mW -> 100kΩ ±1% 62.5mW; footprint UNI_ROYAL_0402WGF3302TCE:R0402 -> UNI_ROYAL_0402WGF1003TCE:R0402
- U3: value 10µH ±20% -> (none)
Connections:
- net SW renamed cathode
- net VIN renamed nSHDN
- C2 pad 2: regulator-gnd-1 -> regulator-gnd
- C3 pad 2: regulator-gnd -> regulator-gnd-1
- R1 pad 2: regulator-gnd -> regulator-gnd-1

Commit message: add build_all.py
Parts:
- R1: value 30kΩ ±1% 62.5mW -> 10kΩ ±1% 62.5mW; footprint UNI_ROYAL_0402WGF3002TCE:R0402 -> UNI_ROYAL_0402WGF1002TCE:R0402
- R2: value 100kΩ ±1% 62.5mW -> 33kΩ ±1% 62.5mW; footprint UNI_ROYAL_0402WGF1003TCE:R0402 -> UNI_ROYAL_0402WGF3302TCE:R0402
Connections:
- net cathode renamed SW
- net nSHDN renamed VIN
Changed lines of the file:
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@@
     (net 7 "regulator.ic.footprint.pins[1].net-net")
     (net 8 "regulator.ic.footprint.pins[2].net-net")
-    (net 9 "nSHDN")
+    (net 9 "VIN")
     (net 10 "regulator.ic.footprint.pins[5].net-net")
     (net 11 "regulator.ic.footprint.pins[0].net-net")
     (net 12 "regulator.ic.footprint.pins[4].net-net")
     (net 13 "regulator-gnd")
-    (net 14 "cathode")
+    (net 14 "SW")
     (net 15 "regulator.inductor.footprint.pins[1].net-net")
     (footprint "CCTC_TCC0402X5R474M160AT:C0402"
@@
             (size 0.79 0.54)
             (layers "F.Cu" "F.Paste" "F.Mask")
-            (net 14 "cathode")
+            (net 14 "SW")
         )
         (pad "1" smd rect
@@
             (size 1.41 1.35)
             (layers "F.Cu" "F.Paste" "F.Mask")
-            (net 9 "nSHDN")
+            (net 9 "VIN")
         )
         (model "${KIPRJMOD}/../../parts/SAMSUNG_CL21A475KAQNNNE/C0805_L2.0-W1.3-H1.3.step"
@@
         )
     )
-    (footprint "UNI_ROYAL_0402WGF3002TCE:R0402"
+    (footprint "UNI_ROYAL_0402WGF1002TCE:R0402"
         (layer "F.Cu")
         (at 10 0 0)
@@
             )
         )
-        (property "Value" "30kΩ ±1% 62.5mW"
+        (property "Value" "10kΩ ±1% 62.5mW"
             (at 0 4 0)
             (layer "F.Fab")
@@
             )
         )
-        (property "__atopile_lib_fp_hash__" "05c9e6f4-6f44-8e4c-3936-bdd66f768132"
-            (at 0 0 0)
-            (layer "User.9")
-            (hide yes)
-            (effects
-                (font
-                    (size 0.125 0.125)
-                    (thickness 0.01875)
-                )
-            )
-        )
-        (property "LCSC" "C25776"
-            (at 0 0 0)
-            (layer "User.9")
-            (hide yes)
-            (effects
-                (font
-                    (size 0.125 0.125)
-                    (thickness 0.01875)
-                )
-            )
-        )
-        (property "Partnumber" "0402WGF3002TCE"
+        (property "__atopile_lib_fp_hash__" "52234549-8985-85d4-dd79-0d66742cf16c"
+            (at 0 0 0)
+            (layer "User.9")
+            (hide yes)
+            (effects
+                (font
+                    (size 0.125 0.125)
+                    (thickness 0.01875)
+                )
+            )
+        )
+        (property "LCSC" "C25744"
+            (at 0 0 0)
+            (layer "User.9")
+            (hide yes)
+            (effects
+                (font
+                    (size 0.125 0.125)
+                    (thickness 0.01875)
+                )
+            )
+        )
+        (property "Partnumber" "0402WGF1002TCE"
             (at 0 0 0)
             (layer "User.9")
@@
             )
         )
-        (property "PARAM_resistance" "{\"type\": \"Quantity_Interval_Disjoint\", \"data\": {\"intervals\": {\"type\": \"Numeric_Interval_Disjoint\", \"data\": {\"intervals\": [{\"type\": \"Numeric_Interval\", \"data\": {\"min\": 29700.000006705523, \"max\": 30299.999993294477}}]}}, \"unit\": \"ohm\"}}"
+        (property "PARAM_resistance" "{\"type\": \"Quantity_Interval_Disjoint\", \"data\": {\"intervals\": {\"type\": \"Numeric_Interval_Disjoint\", \"data\": {\"intervals\": [{\"type\": \"Numeric_Interval\", \"data\": {\"min\": 9900.000002235174, \"max\": 10099.999997764826}}]}}, \"unit\": \"ohm\"}}"
             (at 0 0 0)
             (layer "User.9")
@@
             )
         )
-        (property "checksum" "aec7d2e7474626b8b90b690d4366d48d116d55b95a44e6664ebbf5b41d6fcb2a"
+        (property "checksum" "259c8f2b3c4ed145b90b418853b1dc377fc6c3fd12e0e8205ed5f17f665dfda4"
             (at 0 0 0)
             (layer "User.9")
@@
             )
         )
-        (property "Datasheet" "https://www.lcsc.com/datasheet/lcsc_datasheet_2206010100_UNI-ROYAL-Uniroyal-Elec-0402WGF3002TCE_C25776.pdf"
+        (property "Datasheet" "https://www.lcsc.com/datasheet/lcsc_datasheet_2411221126_UNI-ROYAL-Uniroyal-Elec-0402WGF1002TCE_C25744.pdf"
             (at 0 0 0)
             (layer "User.9")
@@
             (net 2 "FB")
         )
-        (model "${KIPRJMOD}/../../parts/UNI_ROYAL_0402WGF3002TCE/R0402_L1.0-W0.5-H0.4.step"
+        (model "${KIPRJMOD}/../../parts/UNI_ROYAL_0402WGF1002TCE/R0402_L1.0-W0.5-H0.4.step"
             (offset
                 (xyz 0 0 0)
@@
         )
     )
-    (footprint "UNI_ROYAL_0402WGF1003TCE:R0402"
+    (footprint "UNI_ROYAL_0402WGF3302TCE:R0402"
         (layer "F.Cu")
         (at 10 -10 0)
@@
             )
         )
-        (property "Value" "100kΩ ±1% 62.5mW"
+        (property "Value" "33kΩ ±1% 62.5mW"
             (at 0 4 0)
             (layer "F.Fab")
@@
             )
         )
-        (property "__atopile_lib_fp_hash__" "e9a34ec6-a8b0-5db1-089e-339c9c470f59"
-            (at 0 0 0)
-            (layer "User.9")
-            (hide yes)
-            (effects
-                (font
-                    (size 0.125 0.125)
-                    (thickness 0.01875)
-                )
-            )
-        )
-        (property "LCSC" "C25741"
-            (at 0 0 0)
-            (layer "User.9")
-            (hide yes)
-            (effects
-                (font
-                    (size 0.125 0.125)
-                    (thickness 0.01875)
-                )
-            )
-        )
-        (property "Partnumber" "0402WGF1003TCE"
+        (property "__atopile_lib_fp_hash__" "d1db4d1f-8259-a6eb-c308-48ec2789f4ec"
+            (at 0 0 0)
+            (layer "User.9")
+            (hide yes)
+            (effects
+                (font
+                    (size 0.125 0.125)
+                    (thickness 0.01875)
+                )
+            )
+        )
+        (property "LCSC" "C25779"
+            (at 0 0 0)
+            (layer "User.9")
+            (hide yes)
+            (effects
+                (font
+                    (size 0.125 0.125)
+                    (thickness 0.01875)
+                )
+            )
+        )
+        (property "Partnumber" "0402WGF3302TCE"
             (at 0 0 0)
             (layer "User.9")
@@
             )
         )
-        (property "PARAM_resistance" "{\"type\": \"Quantity_Interval_Disjoint\", \"data\": {\"intervals\": {\"type\": \"Numeric_Interval_Disjoint\", \"data\": {\"intervals\": [{\"type\": \"Numeric_Interval\", \"data\": {\"min\": 99000.00002235174, \"max\": 100999.99997764826}}]}}, \"unit\": \"ohm\"}}"
+        (property "PARAM_resistance" "{\"type\": \"Quantity_Interval_Disjoint\", \"data\": {\"intervals\": {\"type\": \"Numeric_Interval_Disjoint\", \"data\": {\"intervals\": [{\"type\": \"Numeric_Interval\", \"data\": {\"min\": 32670.000007376075, \"max\": 33329.999992623925}}]}}, \"unit\": \"ohm\"}}"
             (at 0 0 0)
             (layer "User.9")
@@
             )
         )
-        (property "checksum" "4ef51b9dd8d4109c730b3a8030c276a1ff93a5448dcf057803debc405a07738a"
+        (property "checksum" "2faa9480c22de74657318ea0ec5b82772826c736abc15b259fd3629c5ab0ba5c"
             (at 0 0 0)
             (layer "User.9")
@@
             )
         )
-        (property "Datasheet" "https://www.lcsc.com/datasheet/lcsc_datasheet_2206010100_UNI-ROYAL-Uniroyal-Elec-0402WGF1003TCE_C25741.pdf"
+        (property "Datasheet" "https://www.lcsc.com/datasheet/lcsc_datasheet_2206010100_UNI-ROYAL-Uniroyal-Elec-0402WGF3302TCE_C25779.pdf"
             (at 0 0 0)
             (layer "User.9")
@@
             (net 4 "hv")
         )
-        (model "${KIPRJMOD}/../../parts/UNI_ROYAL_0402WGF1003TCE/R0402_L1.0-W0.5-H0.4.step"
+        (model "${KIPRJMOD}/../../parts/UNI_ROYAL_0402WGF3302TCE/R0402_L1.0-W0.5-H0.4.step"
             (offset
                 (xyz 0 0 0)

Commit message: update ti-lv28 layout
Parts:
- added D1: , Hottech_1N5819WS:SOD-323_L1.8-W1.3-LS2.5-RD, F.Cu at (0.00, 0.00)
- C2: footprint SAMSUNG_CL21A475KAQNNNE:C0805 -> Samsung_Electro_Mechanics_CL21A475KAQNNNE:C0805
- C3: footprint SAMSUNG_CL21A106KAYNNNE:C0805 -> Samsung_Electro_Mechanics_CL21A106KAYNNNE:C0805
Connections:
- net regulator.inductor.footprint.pins[0].net-net renamed regulator.inductor-net-1
- net regulator.inductor.footprint.pins[1].net-net renamed regulator.inductor-net
- C1 pad 2: SW -> cathode
- C2 pad 1: VIN -> nSHDN
- C2 pad 2: regulator-gnd -> regulator-gnd-1
- C3 pad 2: regulator-gnd-1 -> regulator-gnd
- R1 pad 2: regulator-gnd-1 -> regulator-gnd
- U2 pad 1: regulator.ic.footprint.pins[0].net-net -> CB
- U2 pad 2: regulator.ic.footprint.pins[1].net-net -> regulator-gnd-1
- U2 pad 3: regulator.ic.footprint.pins[2].net-net -> FB
- U2 pad 4: regulator.ic.footprint.pins[3].net-net -> nSHDN
- U2 pad 5: regulator.ic.footprint.pins[4].net-net -> nSHDN
- U2 pad 6: regulator.ic.footprint.pins[5].net-net -> cathode
