File: packages/stemma_connectors/layouts/example/example.kicad_pcb (KiCad board)
At the start: 2 copper layers, 10 x 10 mm, 1 part

Commit message: layout
Parts:
- moved CN1 181.4 mm to (0.00, 0.00)

Commit message: layout 2
Parts:
- moved CN1 181.2 mm to (150.0, 101.7)

Commit message: rebuild again
Connections:
- net line renamed -line-0
- net line-1 renamed -line-1
