File: packages/ti-tps54560x/layouts/test-3v3/test-3v3.kicad_pcb (KiCad board)
At the start: 2 copper layers, 17 parts

Commit message: Fix frozen for regulator
Parts:
- R1: value 23.7kΩ ±1% 62.5mW -> 24kΩ ±0% 62.5mW
Connections:
- net cathode renamed SW
- net hv-1 renamed regulator-hv
Changed lines of the file:
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@@
     (net 2 "COMP")
     (net 3 "net")
-    (net 5 "cathode")
+    (net 5 "SW")
     (net 6 "gnd")
     (net 7 "BOOT")
     (net 8 "RT_CLK")
     (net 9 "FB")
-    (net 10 "hv-1")
+    (net 10 "regulator-hv")
     (footprint "atopile:C0805-3b2e55"
         (layer "F.Cu")
@@
             (size 1.41 1.35)
             (layers "F.Cu" "F.Paste" "F.Mask")
-            (net 10 "hv-1")
+            (net 10 "regulator-hv")
         )
     )
@@
             (size 1.41 1.35)
             (layers "F.Cu" "F.Paste" "F.Mask")
-            (net 10 "hv-1")
+            (net 10 "regulator-hv")
         )
     )
@@
             (size 0.79 0.54)
             (layers "F.Cu" "F.Paste" "F.Mask")
-            (net 5 "cathode")
+            (net 5 "SW")
         )
         (pad "1" smd rect
@@
             )
         )
-        (property "Value" "23.7kΩ ±1% 62.5mW"
+        (property "Value" "24kΩ ±0% 62.5mW"
             (at 0 4 0)
             (layer "F.Fab")
@@
             )
         )
-        (property "LCSC" "C327362"
+        (property "LCSC" "C407741"
             (at 0 0 0)
             (layer "User.9")
@@
             )
         )
-        (property "Partnumber" "RC0402FR-0723K7L"
+        (property "Partnumber" "0402WGD2402TCE"
             (at 0 0 0)
             (layer "User.9")
@@
             )
         )
-        (property "Manufacturer" "YAGEO"
+        (property "Manufacturer" "UNI-ROYAL(Uniroyal Elec)"
             (at 0 0 0)
             (layer "User.9")
@@
             )
         )
-        (property "JLCPCB description" "62.5mW Thick Film Resistors 50V ±100ppm/℃ ±1% 23.7kΩ 0402  Chip Resistor - Surface Mount ROHS"
+        (property "JLCPCB description" "62.5mW Thick Film Resistors 50V ±100ppm/℃ ±0.5% 24kΩ 0402  Chip Resistor - Surface Mount ROHS"
             (at 0 0 0)
             (layer "User.9")
@@
             )
         )
-        (property "PARAM_resistance" "{\"type\": \"Quantity_Interval_Disjoint\", \"data\": {\"intervals\": {\"type\": \"Numeric_Interval_Disjoint\", \"data\": {\"intervals\": [{\"type\": \"Numeric_Interval\", \"data\": {\"min\": 23463.000005297363, \"max\": 23936.999994702637}}]}}, \"unit\": \"ohm\"}}"
+        (property "PARAM_resistance" "{\"type\": \"Quantity_Interval_Disjoint\", \"data\": {\"intervals\": {\"type\": \"Numeric_Interval_Disjoint\", \"data\": {\"intervals\": [{\"type\": \"Numeric_Interval\", \"data\": {\"min\": 23880.00000268221, \"max\": 24119.99999731779}}]}}, \"unit\": \"ohm\"}}"
             (at 0 0 0)
             (layer "User.9")
@@
             (size 2.05 2.19)
             (layers "F.Cu" "F.Paste" "F.Mask")
-            (net 5 "cathode")
+            (net 5 "SW")
         )
     )
@@
             (size 0.57 2.04)
             (layers "F.Cu" "F.Paste" "F.Mask")
-            (net 5 "cathode")
+            (net 5 "SW")
         )
         (pad "7" smd oval
@@
             (size 2.92 6.42)
             (layers "F.Cu" "F.Paste" "F.Mask")
-            (net 5 "cathode")
+            (net 5 "SW")
         )
         (pad "2" smd rect
@@
             (size 2.92 6.42)
             (layers "F.Cu" "F.Paste" "F.Mask")
-            (net 10 "hv-1")
+            (net 10 "regulator-hv")
         )
     )
@@
             )
         )
-        (property "LCSC" "C138003"
+        (property "LCSC" "C25779"
             (at 0 0 0)
             (layer "User.9")
@@
             )
         )
-        (property "Partnumber" "RC0402FR-0733KL"
+        (property "Partnumber" "0402WGF3302TCE"
             (at 0 0 0)
             (layer "User.9")
@@
             )
         )
-        (property "Manufacturer" "YAGEO"
+        (property "Manufacturer" "UNI-ROYAL(Uniroyal Elec)"
             (at 0 0 0)
             (layer "User.9")
@@
             )
         )
-        (property "LCSC" "C60491"
+        (property "LCSC" "C25741"
             (at 0 0 0)
             (layer "User.9")
@@
             )
         )
-        (property "Partnumber" "RC0402FR-07100KL"
+        (property "Partnumber" "0402WGF1003TCE"
             (at 0 0 0)
             (layer "User.9")
@@
             )
         )
-        (property "Manufacturer" "YAGEO"
+        (property "Manufacturer" "UNI-ROYAL(Uniroyal Elec)"
             (at 0 0 0)
             (layer "User.9")
@@
             (size 0.57 0.54)
             (layers "F.Cu" "F.Paste" "F.Mask")
-            (net 10 "hv-1")
+            (net 10 "regulator-hv")
         )
     )
@@
             (size 1.41 1.35)
             (layers "F.Cu" "F.Paste" "F.Mask")
-            (net 10 "hv-1")
+            (net 10 "regulator-hv")
         )
     )
@@
             (size 1.41 1.35)
             (layers "F.Cu" "F.Paste" "F.Mask")
-            (net 10 "hv-1")
+            (net 10 "regulator-hv")
         )
     )

Commit message: fix tps54560x compile error
Parts:
- C1: footprint atopile:C0402-b3ef17 -> Samsung_Electro_Mechanics_CL05B104KB54PNC:C0402
- C10, C7, C8, C9: value 22µF ±20% 25V X5R -> 22µF ±20% 35V X5R; footprint atopile:C0805-3b2e55 -> HRE_CGA0805X5R226M350MT:C0805
- C2: footprint atopile:C0402-b3ef17 -> Murata_Electronics_GRM1555C1H472JE01D:C0402
- C3: footprint atopile:C0402-b3ef17 -> Kyocera_AVX_04025A8R2JAT2A:C0402
- C4, C5, C6: footprint atopile:C0805-3b2e55 -> Murata_Electronics_GRM21BR61H106KE43L:C0805
- D1: footprint atopile:SMB_L4.6-W3.6-LS5.3-RD-330cb3 -> ST_STPS340U:SMB_L4.6-W3.6-LS5.3-RD
- L1: footprint atopile:IND-SMD_L8.0-W8.0_SWPA8040S-2a70f8 -> Sunlord_SWPA8040S5R6NT:IND-SMD_L8.0-W8.0_SWPA8040S
- R1: value 24kΩ ±0% 62.5mW -> 23.7kΩ ±1% 62.5mW; footprint atopile:R0402-56259e -> YAGEO_RC0402FR_0723K7L:R0402
- R2: footprint atopile:R0402-56259e -> UNI_ROYAL_0402WGF3302TCE:R0402
- R3: footprint atopile:R0402-56259e -> UNI_ROYAL_0402WGF1003TCE:R0402
- R4: footprint atopile:R0402-56259e -> UNI_ROYAL_0402WGF1623TCE:R0402
- U1: footprint atopile:SOIC-8_L5.0-W4.0-P1.27-LS6.0-BL-EP2.0-748c0f -> TI_TPS54560DDAR:SOIC-8_L5.0-W4.0-P1.27-LS6.0-BL-EP2.0
Connections:
- net SW renamed cathode
- net net renamed regulator-net
- U1 pad : (no net) -> regulator.ic.footprint.pins[0].net-net

Commit message: add build_all.py
Connections:
- net cathode renamed SW
Changed lines of the file:
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@@
     (net 2 "COMP")
     (net 3 "regulator-net")
-    (net 5 "cathode")
+    (net 5 "SW")
     (net 6 "gnd")
     (net 7 "BOOT")
@@
             (size 0.79 0.54)
             (layers "F.Cu" "F.Paste" "F.Mask")
-            (net 5 "cathode")
+            (net 5 "SW")
         )
         (pad "1" smd rect
@@
             (size 2.05 2.19)
             (layers "F.Cu" "F.Paste" "F.Mask")
-            (net 5 "cathode")
+            (net 5 "SW")
         )
         (model "${KIPRJMOD}/../../parts/ST_STPS340U/SMB_L4.6-W3.6-LS5.3-RD.step"
@@
             (size 0.57 2.04)
             (layers "F.Cu" "F.Paste" "F.Mask")
-            (net 5 "cathode")
+            (net 5 "SW")
         )
         (pad "7" smd oval
@@
             )
         )
-        (property "__atopile_lib_fp_hash__" "e0b990ef-fe82-e3b8-fc10-7c8fdd6b5159"
+        (property "__atopile_lib_fp_hash__" "71edee91-115f-cefb-5024-526b55d8a9aa"
             (at 0 0 0)
             (layer "User.9")
@@
             )
         )
-        (property "checksum" "72ce702531c80bc8c33ea3b1f5174c7763c47f97a929ccd9fa5530b7692d9152"
+        (property "checksum" "18155deb31f646a6d966b493cdb3c0eab4e2378502c1e5b1c52c5155c8b331be"
             (at 0 0 0)
             (layer "User.9")
@@
             (size 2.92 6.42)
             (layers "F.Cu" "F.Paste" "F.Mask")
-            (net 5 "cathode")
+            (net 5 "SW")
         )
         (pad "2" smd rect
@@
             (net 10 "regulator-hv")
         )
-        (model "${KIPRJMOD}/../../build/cache/parts/easyeda/C96972/IND-SMD_L8.0-W8.0-H4.2.step"
+        (model "${KIPRJMOD}/../../parts/Sunlord_SWPA8040S5R6NT/IND-SMD_L8.0-W8.0-H4.2.STEP"
             (offset
                 (xyz 0 0 0)

Commit message: update with 3d models
Parts:
- C10, C7, C8, C9: value 22µF ±20% 35V X5R -> 22µF ±20% 25V X5R; footprint HRE_CGA0805X5R226M350MT:C0805 -> Samsung_Electro_Mechanics_CL21A226MAQNNNE:C0805
- D1: footprint ST_STPS340U:SMB_L4.6-W3.6-LS5.3-RD -> STMicroelectronics_STPS340U:SMB_L4.6-W3.6-LS5.3-RD
- U1: footprint TI_TPS54560DDAR:SOIC-8_L5.0-W4.0-P1.27-LS6.0-BL-EP2.0 -> Texas_Instruments_TPS54560DDAR:SOIC-8_L5.0-W4.0-P1.27-LS6.0-BL-EP2.0
Connections:
- net SW renamed cathode

Commit message: update tps54560
Connections:
- net cathode renamed SW

Commit message: chore: Update packages for ato 0.10.7 (#69)
- Updates layouts with new net names due to https://github.com/atopile/atopile/pull/1226
- Disables failing DRCs
  - TODO: fix and re-enable for example/test/reference design builds that should be complete
  - TODO: make DRCs configurable and be more selective about what's disabled for "library" packages
Connections:
- net SW renamed cathode
- net hv renamed -hv
Changed lines of the file:
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@@
     )
     (net 0 "")
-    (net 1 "hv")
+    (net 1 "-hv")
     (net 2 "COMP")
     (net 3 "regulator-net")
-    (net 5 "SW")
+    (net 5 "cathode")
     (net 6 "gnd")
     (net 7 "BOOT")
@@
             )
         )
-        (property "__atopile_lib_fp_hash__" "77114461-70c2-b27a-938f-42c1a972c1d2"
+        (property "__atopile_lib_fp_hash__" "0ef0838e-a0a0-0bdb-24b7-004799b4e846"
             (at 0 0 0)
             (layer "User.9")
@@
             )
         )
-        (property "checksum" "eff7ad33620499c4e3b6cee6ca4f0577458a2817743f120dd7491af73fc3650a"
+        (property "checksum" "f94349e09ab29468f9c2eb4a152973fa23f3222215254540c17f0ab71bf55e30"
             (at 0 0 0)
             (layer "User.9")
@@
             (size 1.41 1.35)
             (layers "F.Cu" "F.Paste" "F.Mask")
-            (net 1 "hv")
+            (net 1 "-hv")
         )
         (model "${KIPRJMOD}/../../parts/Murata_Electronics_GRM21BR61H106KE43L/C0805_L2.0-W1.3-H1.3.step"
@@
             )
         )
-        (property "__atopile_lib_fp_hash__" "efa7a6da-feac-0f08-6721-2bf885b18f95"
+        (property "__atopile_lib_fp_hash__" "bcac8612-6069-3884-f91e-c4a397778bb3"
             (at 0 0 0)
             (layer "User.9")
@@
             )
         )
-        (property "checksum" "e0cceabcbd4745ac32546fe02bcdb40717aee495041a61cc242c7ac8f2de136c"
+        (property "checksum" "7761f8589b1326c829d2a20c84d27ce2768a4f0e98efb35f5f2bd4c79034cbf2"
             (at 0 0 0)
             (layer "User.9")
@@
             )
         )
-        (property "__atopile_lib_fp_hash__" "efa7a6da-feac-0f08-6721-2bf885b18f95"
+        (property "__atopile_lib_fp_hash__" "bcac8612-6069-3884-f91e-c4a397778bb3"
             (at 0 0 0)
             (layer "User.9")
@@
             )
         )
-        (property "checksum" "e0cceabcbd4745ac32546fe02bcdb40717aee495041a61cc242c7ac8f2de136c"
+        (property "checksum" "7761f8589b1326c829d2a20c84d27ce2768a4f0e98efb35f5f2bd4c79034cbf2"
             (at 0 0 0)
             (layer "User.9")
@@
             )
         )
-        (property "__atopile_lib_fp_hash__" "61a94387-919d-9941-de7f-607166db09b0"
+        (property "__atopile_lib_fp_hash__" "70b8cd38-9be2-35ce-a4c7-1fb71b20b8f3"
             (at 0 0 0)
             (layer "User.9")
@@
             )
         )
-        (property "checksum" "f41d7593e1df2cbf7f789d139c6aacf1d28714c28a6c550f9340ea4175556621"
+        (property "checksum" "8ae8b38ca4b30c8413b05faba0581c3f2241f00897bddd49775f59afcc646643"
             (at 0 0 0)
             (layer "User.9")
@@
             (size 0.79 0.54)
             (layers "F.Cu" "F.Paste" "F.Mask")
-            (net 5 "SW")
+            (net 5 "cathode")
         )
         (pad "1" smd rect
@@
             )
         )
-        (property "__atopile_lib_fp_hash__" "76170170-d69a-2eae-9563-f25625bb7bd3"
+        (property "__atopile_lib_fp_hash__" "f806a0a6-fb7d-3e68-a522-5269ffacbe2d"
             (at 0 0 0)
             (layer "User.9")
@@
             )
         )
-        (property "checksum" "dddc6432e3c179677b6f88115e10ec8fc6f5ce19ae80386549922efd3e4c264d"
+        (property "checksum" "7800b16fbe92d14fb1bd1c66586cdda7609ccbb29113cf6faeb6b3f43bac4b31"
             (at 0 0 0)
             (layer "User.9")
@@
             )
         )
-        (property "__atopile_lib_fp_hash__" "74b05314-9f93-c6a3-20a8-3fe48abed109"
+        (property "__atopile_lib_fp_hash__" "6b06e7af-6c6f-02f8-2ae6-fa8636a32d32"
             (at 0 0 0)
             (layer "User.9")
@@
             )
         )
-        (property "checksum" "60332310227e1cd04c8db6f8ac2f14b294e7a0632f51db921f5f221d0a9cf168"
+        (property "checksum" "6b26152d9d5b211281fa8f7302d4bbc962ca71e7da7a227c557d557ff1936f19"
             (at 0 0 0)
             (layer "User.9")
@@
             (size 2.05 2.19)
             (layers "F.Cu" "F.Paste" "F.Mask")
-            (net 5 "SW")
+            (net 5 "cathode")
         )
         (model "${KIPRJMOD}/../../parts/STMicroelectronics_STPS340U/SMB_L4.6-W3.6-LS5.3-RD.step"
@@
             )
         )
-        (property "__atopile_lib_fp_hash__" "7bd5e56d-cc4e-c053-8ebd-6587558e6182"
+        (property "__atopile_lib_fp_hash__" "fca1a759-150e-fdad-e063-cf90b1064e89"
             (at 0 0 0)
             (layer "User.9")
@@
             )
         )
-        (property "checksum" "b6c9e31e180bec60ae51ffdef13110badddf1ba1b71bea51ce76b34f582758c3"
+        (property "checksum" "57820cacbecd9b139e925ad71cbd9392b38a38fb4baa5264277f1590a1f3b86d"
             (at 0 0 0)
             (layer "User.9")
@@
             (size 0.57 2.04)
             (layers "F.Cu" "F.Paste" "F.Mask")
-            (net 1 "hv")
+            (net 1 "-hv")
         )
         (pad "3" smd oval
@@
             (size 0.57 2.04)
             (layers "F.Cu" "F.Paste" "F.Mask")
-            (net 1 "hv")
+            (net 1 "-hv")
         )
         (pad "4" smd oval
@@
             (size 0.57 2.04)
             (layers "F.Cu" "F.Paste" "F.Mask")
-            (net 5 "SW")
+            (net 5 "cathode")
         )
         (pad "7" smd oval
@@
             (size 2.92 6.42)
             (layers "F.Cu" "F.Paste" "F.Mask")
-            (net 5 "SW")
+            (net 5 "cathode")
         )
         (pad "2" smd rect
@@
             )
         )
-        (property "__atopile_lib_fp_hash__" "77114461-70c2-b27a-938f-42c1a972c1d2"
+        (property "__atopile_lib_fp_hash__" "0ef0838e-a0a0-0bdb-24b7-004799b4e846"
             (at 0 0 0)
             (layer "User.9")
@@
             )
         )
-        (property "checksum" "eff7ad33620499c4e3b6cee6ca4f0577458a2817743f120dd7491af73fc3650a"
+        (property "checksum" "f94349e09ab29468f9c2eb4a152973fa23f3222215254540c17f0ab71bf55e30"
             (at 0 0 0)
             (layer "User.9")
@@
             (size 1.41 1.35)
             (layers "F.Cu" "F.Paste" "F.Mask")
-            (net 1 "hv")
+            (net 1 "-hv")
         )
         (model "${KIPRJMOD}/../../parts/Murata_Electronics_GRM21BR61H106KE43L/C0805_L2.0-W1.3-H1.3.step"
@@
             )
         )
-        (property "__atopile_lib_fp_hash__" "77114461-70c2-b27a-938f-42c1a972c1d2"
+        (property "__atopile_lib_fp_hash__" "0ef0838e-a0a0-0bdb-24b7-004799b4e846"
             (at 0 0 0)
             (layer "User.9")
@@
             )
         )
-        (property "checksum" "eff7ad33620499c4e3b6cee6ca4f0577458a2817743f120dd7491af73fc3650a"
+        (property "checksum" "f94349e09ab29468f9c2eb4a152973fa23f3222215254540c17f0ab71bf55e30"
             (at 0 0 0)
             (layer "User.9")
@@
             (size 1.41 1.35)
             (layers "F.Cu" "F.Paste" "F.Mask")
-            (net 1 "hv")
+            (net 1 "-hv")
         )
         (model "${KIPRJMOD}/../../parts/Murata_Electronics_GRM21BR61H106KE43L/C0805_L2.0-W1.3-H1.3.step"
@@
             )
         )
-        (property "__atopile_lib_fp_hash__" "383cf47f-dc4e-610f-aa15-96fc8c890bc8"
+        (property "__atopile_lib_fp_hash__" "ccdb8997-a62b-1028-934d-b0f22ce30324"
             (at 0 0 0)
             (layer "User.9")
@@
             )
         )
-        (property "checksum" "05135ae40f8c2fd44f2e7f4d1b742c2b91d16bf599220632b7d7cef727cbc5a4"
+        (property "checksum" "36c0051bacd408f5bc69d43d751a0b7ed810432a91edb9cb9d2d68d585af84ba"
             (at 0 0 0)
             (layer "User.9")
@@
             )
         )
-        (property "__atopile_lib_fp_hash__" "7e791553-8c7c-5c13-e2ad-3c559fc6973e"
+        (property "__atopile_lib_fp_hash__" "351ae59c-4aae-5053-4369-421b3f5dcc43"
             (at 0 0 0)
             (layer "User.9")
@@
             )
         )
-        (property "checksum" "1851a99f7280a693e571bbe3c7db50465001a76950d485e211e7659e23394f80"
+        (property "checksum" "937691df9fbb6fe6614e5a0fc59b7ae294187a1937fefbee26fb3eec544cfa53"
             (at 0 0 0)
             (layer "User.9")
@@
             )
         )
-        (property "__atopile_lib_fp_hash__" "a33aff4c-85c5-7ca6-a74c-f5fc455716f5"
+        (property "__atopile_lib_fp_hash__" "43e99e95-6c29-b9ab-1f6b-185556aed720"
             (at 0 0 0)
             (layer "User.9")
@@
             )
         )
-        (property "checksum" "ea2cc4d64baf06e9b5dabbd663a953df5da362d62d0ae4a3fc276f4682cab789"
+        (property "checksum" "953a23a13dfc937c4f3b37f71aa0121e901b2604e8d18e5d1b04350766e1a21d"
             (at 0 0 0)
             (layer "User.9")
@@
             )
         )
-        (property "__atopile_lib_fp_hash__" "efa7a6da-feac-0f08-6721-2bf885b18f95"
+        (property "__atopile_lib_fp_hash__" "bcac8612-6069-3884-f91e-c4a397778bb3"
             (at 0 0 0)
             (layer "User.9")
@@
             )
         )
-        (property "checksum" "e0cceabcbd4745ac32546fe02bcdb40717aee495041a61cc242c7ac8f2de136c"
+        (property "checksum" "7761f8589b1326c829d2a20c84d27ce2768a4f0e98efb35f5f2bd4c79034cbf2"
             (at 0 0 0)
             (layer "User.9")
@@
             )
         )
-        (property "__atopile_lib_fp_hash__" "efa7a6da-feac-0f08-6721-2bf885b18f95"
+        (property "__atopile_lib_fp_hash__" "bcac8612-6069-3884-f91e-c4a397778bb3"
             (at 0 0 0)
             (layer "User.9")
@@
             )
         )
-        (property "checksum" "e0cceabcbd4745ac32546fe02bcdb40717aee495041a61cc242c7ac8f2de136c"
+        (property "checksum" "7761f8589b1326c829d2a20c84d27ce2768a4f0e98efb35f5f2bd4c79034cbf2"
             (at 0 0 0)
             (layer "User.9")
