File: packages/st-lsm6ds3tr-c/layouts/usage/usage.kicad_pcb (KiCad board)
At the start: 2 copper layers, 0 parts

Commit message: fix checksum
Parts:
- added C1: 100nF ±10% 16V X7R, Samsung_Electro_Mechanics_CL05B104KO5NNNC:C0402, F.Cu at (0.00, -40.0)
- added C2: 100nF ±10% 16V X7R, Samsung_Electro_Mechanics_CL05B104KO5NNNC:C0402, F.Cu at (0.00, -50.0)
- added R1: 10kΩ ±1% 62.5mW, UNI_ROYAL_0402WGF1002TCE:R0402, F.Cu at (0.00, 0.00)
- added R2: 10kΩ ±1% 62.5mW, UNI_ROYAL_0402WGF1002TCE:R0402, F.Cu at (0.00, -10.0)
- added R3: 10kΩ ±1% 62.5mW, UNI_ROYAL_0402WGF1002TCE:R0402, F.Cu at (0.00, -20.0)
- added U1: , STMicroelectronics_LSM6DS3TR_C:LGA-14_L3.0-W2.5-P0.50-TL, F.Cu at (0.00, -30.0)
