File: packages/st-lsm6ds3tr-c/layouts/usage/usage.kicad_pcb (KiCad board)
At the start: 2 copper layers, 6 parts

Commit message: st-lsm6ds3tr-c: LLM Update with 0.12.4
Updated st-lsm6ds3tr-c package to work with atopile compiler version 0.12.4.

Changes made:
- Updated requires-atopile from ^0.10.8 to ^0.12.4
- Updated package version from 0.1.0 to 0.1.1
- Rebuilt layouts with new compiler (net naming improvements)
- All builds pass: ato build, ato build --frozen

🤖 Generated with [Claude Code](https://claude.ai/code)

Co-Authored-By: Claude <noreply@anthropic.com>
Connections:
- net SDO_SA0 renamed address_bit_0
- net gnd renamed GND
- net hv renamed VCC
- net imu.package.footprint.pins[1].net-net renamed footprint-net-0
- net imu.package.footprint.pins[2].net-net renamed footprint-net-1
Changed lines of the file:
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@@
     )
     (net 0 "")
-    (net 1 "imu.package.footprint.pins[2].net-net")
-    (net 2 "gnd")
+    (net 1 "footprint-net-1")
+    (net 2 "GND")
     (net 3 "INT1")
     (net 4 "SCL")
@@
     (net 6 "CS")
     (net 7 "SCx")
-    (net 8 "SDO_SA0")
+    (net 8 "address_bit_0")
     (net 9 "SDA")
-    (net 10 "imu.package.footprint.pins[1].net-net")
+    (net 10 "footprint-net-0")
     (net 11 "INT2")
-    (net 12 "hv")
+    (net 12 "VCC")
     (footprint "UNI_ROYAL_0402WGF1002TCE:R0402"
         (layer "F.Cu")
@@
             )
         )
-        (property "__atopile_lib_fp_hash__" "93c4918c-1d67-c6e6-78b1-963e8c3d0716"
+        (property "__atopile_lib_fp_hash__" "ac993d00-cd2e-9909-323a-aafc825a9032"
             (at 0 0 0)
             (layer "User.9")
@@
         )
         (property "atopile_address" "imu.chip_select_pullup"
+            (at 0 0 0)
+            (layer "User.9")
+            (hide yes)
+            (effects
+                (font
+                    (size 0.125 0.125)
+                    (thickness 0.01875)
+                )
+            )
+        )
+        (property "atopile_subaddresses" "[layouts/default/default.kicad_pcb:chip_select_pullup]"
             (at 0 0 0)
             (layer "User.9")
@@
             (size 0.57 0.54)
             (layers "F.Cu" "F.Paste" "F.Mask")
-            (net 12 "hv")
+            (net 12 "VCC")
         )
         (pad "1" smd rect
@@
             )
         )
-        (property "__atopile_lib_fp_hash__" "93c4918c-1d67-c6e6-78b1-963e8c3d0716"
+        (property "__atopile_lib_fp_hash__" "ac993d00-cd2e-9909-323a-aafc825a9032"
             (at 0 0 0)
             (layer "User.9")
@@
         )
         (property "atopile_address" "imu.i2c_pullups[0]"
+            (at 0 0 0)
+            (layer "User.9")
+            (hide yes)
+            (effects
+                (font
+                    (size 0.125 0.125)
+                    (thickness 0.01875)
+                )
+            )
+        )
+        (property "atopile_subaddresses" "[layouts/default/default.kicad_pcb:i2c_pullups[0]]"
             (at 0 0 0)
             (layer "User.9")
@@
             (size 0.57 0.54)
             (layers "F.Cu" "F.Paste" "F.Mask")
-            (net 12 "hv")
+            (net 12 "VCC")
         )
         (pad "1" smd rect
@@
             )
         )
-        (property "__atopile_lib_fp_hash__" "93c4918c-1d67-c6e6-78b1-963e8c3d0716"
+        (property "__atopile_lib_fp_hash__" "ac993d00-cd2e-9909-323a-aafc825a9032"
             (at 0 0 0)
             (layer "User.9")
@@
         )
         (property "atopile_address" "imu.i2c_pullups[1]"
+            (at 0 0 0)
+            (layer "User.9")
+            (hide yes)
+            (effects
+                (font
+                    (size 0.125 0.125)
+                    (thickness 0.01875)
+                )
+            )
+        )
+        (property "atopile_subaddresses" "[layouts/default/default.kicad_pcb:i2c_pullups[1]]"
             (at 0 0 0)
             (layer "User.9")
@@
             (size 0.57 0.54)
             (layers "F.Cu" "F.Paste" "F.Mask")
-            (net 12 "hv")
+            (net 12 "VCC")
         )
         (pad "1" smd rect
@@
             )
         )
-        (property "__atopile_lib_fp_hash__" "521531c6-2872-7c4d-6bdb-32debb7ef4d4"
+        (property "__atopile_lib_fp_hash__" "de60c8d4-0877-a7b8-7f13-9cd8d37255ce"
             (at 0 0 0)
             (layer "User.9")
@@
         )
         (property "atopile_address" "imu.package"
+            (at 0 0 0)
+            (layer "User.9")
+            (hide yes)
+            (effects
+                (font
+                    (size 0.125 0.125)
+                    (thickness 0.01875)
+                )
+            )
+        )
+        (property "atopile_subaddresses" "[layouts/default/default.kicad_pcb:package]"
             (at 0 0 0)
             (layer "User.9")
@@
             (size 0.68 0.28)
             (layers "F.Cu" "F.Paste" "F.Mask")
-            (net 8 "SDO_SA0")
+            (net 8 "address_bit_0")
         )
         (pad "2" smd rect
@@
             (size 0.28 0.68)
             (layers "F.Cu" "F.Paste" "F.Mask")
-            (net 12 "hv")
+            (net 12 "VCC")
         )
         (pad "6" smd rect
@@
             (size 0.28 0.68)
             (layers "F.Cu" "F.Paste" "F.Mask")
-            (net 2 "gnd")
+            (net 2 "GND")
         )
         (pad "7" smd rect
@@
             (size 0.28 0.68)
             (layers "F.Cu" "F.Paste" "F.Mask")
-            (net 2 "gnd")
+            (net 2 "GND")
         )
         (pad "8" smd rect
@@
             (size 0.68 0.28)
             (layers "F.Cu" "F.Paste" "F.Mask")
-            (net 12 "hv")
+            (net 12 "VCC")
         )
         (pad "9" smd rect
@@
             (size 0.68 0.28)
             (layers "F.Cu" "F.Paste" "F.Mask")
-            (net 10 "imu.package.footprint.pins[1].net-net")
+            (net 10 "footprint-net-0")
         )
         (pad "11" smd rect
@@
             (size 0.68 0.28)
             (layers "F.Cu" "F.Paste" "F.Mask")
-            (net 1 "imu.package.footprint.pins[2].net-net")
+            (net 1 "footprint-net-1")
         )
         (pad "12" smd rect
@@
             )
         )
-        (property "__atopile_lib_fp_hash__" "e0f54cc9-1e7d-9688-e09d-ca5527107687"
+        (property "__atopile_lib_fp_hash__" "f8a97365-7255-729e-24e5-6102db053d76"
             (at 0 0 0)
             (layer "User.9")
@@
         )
         (property "atopile_address" "imu.power_caps[0]"
+            (at 0 0 0)
+            (layer "User.9")
+            (hide yes)
+            (effects
+                (font
+                    (size 0.125 0.125)
+                    (thickness 0.01875)
+                )
+            )
+        )
+        (property "atopile_subaddresses" "[layouts/default/default.kicad_pcb:power_caps[0]]"
             (at 0 0 0)
             (layer "User.9")
@@
             (size 0.79 0.54)
             (layers "F.Cu" "F.Paste" "F.Mask")
-            (net 2 "gnd")
+            (net 2 "GND")
         )
         (pad "1" smd rect
@@
             (size 0.79 0.54)
             (layers "F.Cu" "F.Paste" "F.Mask")
-            (net 12 "hv")
+            (net 12 "VCC")
         )
         (model "${KIPRJMOD}/../../parts/Samsung_Electro_Mechanics_CL05B104KO5NNNC/C0402_L1.0-W0.5-H0.5.step"
@@
             )
         )
-        (property "__atopile_lib_fp_hash__" "e0f54cc9-1e7d-9688-e09d-ca5527107687"
+        (property "__atopile_lib_fp_hash__" "f8a97365-7255-729e-24e5-6102db053d76"
             (at 0 0 0)
             (layer "User.9")
@@
         )
         (property "atopile_address" "imu.power_caps[1]"
+            (at 0 0 0)
+            (layer "User.9")
+            (hide yes)
+            (effects
+                (font
+                    (size 0.125 0.125)
+                    (thickness 0.01875)
+                )
+            )
+        )
+        (property "atopile_subaddresses" "[layouts/default/default.kicad_pcb:power_caps[1]]"
             (at 0 0 0)
             (layer "User.9")
@@
             (size 0.79 0.54)
             (layers "F.Cu" "F.Paste" "F.Mask")
-            (net 2 "gnd")
+            (net 2 "GND")
         )
         (pad "1" smd rect
@@
             (size 0.79 0.54)
             (layers "F.Cu" "F.Paste" "F.Mask")
-            (net 12 "hv")
+            (net 12 "VCC")
         )
         (model "${KIPRJMOD}/../../parts/Samsung_Electro_Mechanics_CL05B104KO5NNNC/C0402_L1.0-W0.5-H0.5.step"
@@
         )
     )
+    (group "imu"
+        (members "22db8ba4-bd53-4866-8674-e6514642524b" "5e2506e4-f2a7-441e-b90f-86864642524b" "bf690efa-62f3-478c-91b5-d3aa4642524b" "451861ba-f5ac-4c0a-8ca5-c8b64642524b" "6db09e2f-1429-4103-9c53-e77f4642524b" "1419639d-b096-4b22-b142-13d54642524b")
+    )
 )
