File: packages/ti-ina238/layouts/usage/usage.kicad_pcb (KiCad board)
At the start: 2 copper layers, 3 parts

Commit message: Adafruit Heist 2.0 (#79)
* notes to cursor

* fix CLAUDE.md file referencing

* tidy up ti-ina238

* tidy up MPU6050

* st-lis3mdl

* memsic-mmc5603

* add lis2mdl package

* adi-ds2482s-800: init

* Rule update

* Add TI INA237

* ti-ina3221

* ti-hdc3022

* vishay-vcnl4020

* microchip-24lc32: create

* st-h3lis331: create

* st-lsm6ds3: create

* st-lsm303ag: create

* st-vl53l4cd: create

* st-vl53l4cx: create

* st-lsm303ag: fix drc skip

* vishay-vcnl4200

* bosch-bme688: init

* maxim-ds2484

* skip drc in rule ato.yaml

* AMS TSL2591

* refix instructions

* create st-lsm6dsox

* VCNL4040

* Instr: power first

* liteon-ltr329: create

* liteon-ltr303: create

* liteon-ltr390uv: create

* st-lsm9ds1: init

* ti-dac6578: create

* create bme680

* update VCNL4040

* create microchip-mcp9808

* nxp-pct2075: init

* issi-is31fl3731: create

* MAX17048

* create microchip-mcp9601

* INA237 layout

* infineon-dps310: create

* create microchip-emc2101

* update mcp9808 readme

* MCP4728

* AMS TSL2591

* maxim-ds3231: create

* use arrays

* TCA-8418

* create nxp-pcf8574

* adi-ltc4311

* remove pin info from pcf8574 readme

* remove ada from ato yaml

* aosong-aht20

* ST_LSM6DS3TR_C

* switch chip in nxp-pcf8574

* awinic-aw9523

* switch chip in nxp-pcf8574 usage

* sensirion-sen6x: create

* update bosch-bme280

* create nxp-pcf8575

* bosch-bmp280

* ADI_AD5693R

* bosch-bmp388

* ST_HTS221

* create ti-ads7830

* diodes-inc-74lvc1t45w

* update mpu6050

* maxim-ds3502: create

* switch logic to signal in adc

* microchip-24lc32

* create mcp3421

* maxim-ds1841: create

* microchip-cap1188

* sparkfun-qwiic: create

* invensense-icm20948

* memsic-mmc5603

* update cap1188

* update microchip-mcp23017

* opsco-sk6805-ec15

* opsco-sk6805-ec20

* opsco-sk6805-side

* Sensirion-scd41

* sensirion-sgp40

* update sensirion-sht31

* update sensirion-sht40

* sensirion sht41

* sensirion-sht45

* update rohm-bh1750

* st-ism330dhcx

* st-lis3dh

* st-lps22

* s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
Parts:
- added R2: 10kΩ ±1% 62.5mW, UNI_ROYAL_0402WGF1002TCE:R0402, F.Cu at (0.00, 0.00)
- added R3: 10kΩ ±1% 62.5mW, UNI_ROYAL_0402WGF1002TCE:R0402, F.Cu at (0.00, -10.0)
- R1: value 15mΩ ±1% 1W -> 15mΩ ±1% 250mW; footprint TA_I_Tech_RLM12FTCMR015:RES-SMD_L3.2-W1.6_SY1206 -> Milliohm_HoRF1206_1_4W_15mR_1:R1206
- moved R1 4.34 mm to (148.2, 96.7), turned to -90 degrees
- moved C1 0.30 mm to (152.0, 93.0)
Connections:
- U1 pad 1: gnd -> A1
- U1 pad 2: gnd -> A0
Routing:
- net hv: track 6.27 -> 0.00 mm, vias 1 -> 0
- net (no net): track 0.00 -> 5.28 mm, vias 0 -> 1
- net INneg: track 2.14 -> 5.50 mm
- net gnd: track 4.25 -> 2.33 mm, vias 2 -> 1
