File: packages/adi-ad1938/layouts/example/example.kicad_pcb (KiCad board)
At the start: 2 copper layers, 16 parts

Commit message: Add dockstrings and doc files
Parts:
- added R2: 100kΩ ±1% 62.5mW, UNI_ROYAL_0402WGF1003TCE:R0402, F.Cu at (1.75, 6.75)
- C3, C4: value 10µF ±10% 25V X5R -> 10µF ±10% 16V X5R; footprint Samsung_Electro_Mechanics_CL21A106KAYNNNE:C0805 -> Samsung_Electro_Mechanics_CL21A106KOQNNNE:C0805
Routing:
- net nPD_nRST: track 0.00 -> 2.07 mm, vias 0 -> 1
