File: packages/adi-adbms6830/layouts/input-filters/input-filters.kicad_pcb (KiCad board)
At the start: 2 copper layers, 39 parts

Commit message: trying to build
Parts:
- moved C1 75.7 mm to (30.0, 73.0)
- moved C10 75.7 mm to (120.0, 73.0)
- moved C11 75.7 mm to (130.0, 73.0)
- moved C12 75.7 mm to (140.0, 73.0)
- moved C13 75.7 mm to (150.0, 73.0)
- moved C14 75.7 mm to (160.0, 73.0)
- moved C15 75.7 mm to (170.0, 73.0)
- moved C16 75.7 mm to (180.0, 73.0)
- moved C17 75.7 mm to (190.0, 73.0)
- moved C18 75.7 mm to (200.0, 73.0)
- moved C19 75.7 mm to (210.0, 73.0)
- moved C2 75.7 mm to (40.0, 73.0)
- moved C3 75.7 mm to (50.0, 73.0)
- moved C4 75.7 mm to (60.0, 73.0)
- moved C5 75.7 mm to (70.0, 73.0)
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Other:
- board outline added: 204.9 x 24.1 mm
