File: packages/st-lsm6ds3/layouts/default/default.kicad_pcb (KiCad board)
At the start: 2 copper layers, 7 parts

Commit message: st-lsm6ds3: LLM Update with 0.12.4
Updated st-lsm6ds3 package to work with atopile compiler version 0.12.4.

Changes made:
- Updated requires-atopile from ^0.10.8 to ^0.12.4
- Updated package version from 0.1.0 to 0.1.1
- Rebuilt layouts with new compiler (net naming improvements)
- All builds pass: ato build, ato build --frozen

🤖 Generated with [Claude Code](https://claude.ai/code)

Co-Authored-By: Claude <noreply@anthropic.com>
Connections:
- net gnd renamed GND
- net hv renamed VCC
- net package.footprint.pins[1].net-net renamed footprint-net-0
- net package.footprint.pins[2].net-net renamed footprint-net-1
