File: packages/st-lsm6dsox-lis3mdl/layouts/default/default.kicad_pcb (KiCad board)
At the start: 2 copper layers, 12 parts

Commit message: st-lsm6dsox-lis3mdl: LLM Update with 0.12.4
Updated st-lsm6dsox-lis3mdl package to work with atopile compiler version 0.12.4.

Changes made:
- Updated requires-atopile from ^0.10.8 to ^0.12.4
- Updated package version from 0.1.0 to 0.1.1
- Rebuilt layouts with new compiler (net naming improvements)
- All builds pass: ato build, ato build --frozen

🤖 Generated with [Claude Code](https://claude.ai/code)

Co-Authored-By: Claude <noreply@anthropic.com>
Connections:
- net -CS-0 renamed footprint-CS-0
- net -CS-1 renamed footprint-CS-1
- net SCL_SPC renamed SCL
- net SD0_SA1 renamed lis3mdl_addressor-address_bit_0
- net SDA_SDI_SDO renamed SDA
- net SDO_SA0 renamed lsm6dsox_addressor-address_bit_0
- net gnd renamed GND
- net hv renamed VCC
