File: packages/worldsemi-ws2812c-5050/layouts/default/default.kicad_pcb (KiCad board)
At the start: 2 copper layers, 3 parts

Commit message: Rename pjrc-teensy_4_1 to pjrc-teensy-4-1
- Renamed package directory from pjrc-teensy_4_1 to pjrc-teensy-4-1
- Updated package naming convention to use hyphens instead of underscores
- Package marked as 'Done' in package-todos.md
- Fixed formatting issues (end-of-file and trailing whitespace)
Connections:
- net VDD renamed VCC
- net gnd renamed GND
Changed lines of the file:
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@@
     (net 2 "DOUT")
     (net 3 "line")
-    (net 4 "gnd")
-    (net 5 "VDD")
+    (net 4 "GND")
+    (net 5 "VCC")
     (footprint "Worldsemi_WS2812C:LED-SMD_4P-L5.0-W5.0-LS5.4-TL-1"
         (layer "F.Cu")
@@
             (at 0 0 0)
             (layer "User.9")
-            (hide yes)
-            (effects
-                (font
-                    (size 0.125 0.125)
-                    (thickness 0.01875)
-                )
-            )
-        )
-        (property "__atopile_lib_fp_hash__" "f9538a91-3733-5872-058e-9f49ddf5855e"
+            (hide no)
+            (effects
+                (font
+                    (size 0.125 0.125)
+                    (thickness 0.01875)
+                )
+                (hide yes)
+            )
+        )
+        (property "__atopile_lib_fp_hash__" "48efa57e-110d-c3bd-11fc-3a3a3e43bd40"
             (at 0 0 0)
             (layer "User.9")
@@
         )
         (attr smd)
+        (fp_line
+            (start -2.54 -2.43)
+            (end -2.54 -2.54)
+            (stroke
+                (width 0.25)
+                (type solid)
+            )
+            (layer "F.SilkS")
+        )
+        (fp_line
+            (start -2.54 0.77)
+            (end -2.54 -0.77)
+            (stroke
+                (width 0.25)
+                (type solid)
+            )
+            (layer "F.SilkS")
+        )
+        (fp_line
+            (start 2.54 2.43)
+            (end 2.54 2.54)
+            (stroke
+                (width 0.25)
+                (type solid)
+            )
+            (layer "F.SilkS")
+        )
+        (fp_line
+            (start 2.54 2.54)
+            (end -2.54 2.54)
+            (stroke
+                (width 0.25)
+                (type solid)
+            )
+            (layer "F.SilkS")
+        )
+        (fp_line
+            (start -2.54 2.54)
+            (end -2.54 2.43)
+            (stroke
+                (width 0.25)
+                (type solid)
+            )
+            (layer "F.SilkS")
+        )
+        (fp_line
+            (start 2.54 -0.77)
+            (end 2.54 0.77)
+            (stroke
+                (width 0.25)
+                (type solid)
+            )
+            (layer "F.SilkS")
+        )
         (fp_line
             (start -2.54 -2.54)
@@
         )
         (fp_line
-            (start -2.54 -2.43)
-            (end -2.54 -2.54)
-            (stroke
-                (width 0.25)
-                (type solid)
-            )
-            (layer "F.SilkS")
-        )
-        (fp_line
-            (start -2.54 0.77)
-            (end -2.54 -0.77)
-            (stroke
-                (width 0.25)
-                (type solid)
-            )
-            (layer "F.SilkS")
-        )
-        (fp_line
-            (start -2.54 2.54)
-            (end -2.54 2.43)
-            (stroke
-                (width 0.25)
-                (type solid)
-            )
-            (layer "F.SilkS")
-        )
-        (fp_line
             (start 2.54 -2.54)
             (end 2.54 -2.43)
-            (stroke
-                (width 0.25)
-                (type solid)
-            )
-            (layer "F.SilkS")
-        )
-        (fp_line
-            (start 2.54 -0.77)
-            (end 2.54 0.77)
-            (stroke
-                (width 0.25)
-                (type solid)
-            )
-            (layer "F.SilkS")
-        )
-        (fp_line
-            (start 2.54 2.43)
-            (end 2.54 2.54)
-            (stroke
-                (width 0.25)
-                (type solid)
-            )
-            (layer "F.SilkS")
-        )
-        (fp_line
-            (start 2.54 2.54)
-            (end -2.54 2.54)
             (stroke
                 (width 0.25)
@@
             (layer "F.Fab")
         )
+        (fp_text user "%R"
+            (at 0 0 0)
+            (layer "F.Fab")
+            (effects
+                (font
+                    (size 1 1)
+                    (thickness 0.15)
+                )
+            )
+            (unlocked no)
+        )
         (fp_text user "${REFERENCE}"
             (at 0 -5.65 0)
             (layer "F.SilkS")
-            (hide yes)
-            (effects
-                (font
-                    (size 1 1)
-                    (thickness 0.15)
-                )
-                (hide yes)
-            )
-            (unlocked no)
-        )
-        (fp_text user "${REFERENCE}"
-            (at 0 0 0)
-            (layer "F.Fab")
-            (hide yes)
             (effects
                 (font
@@
             (at -2.35 -1.65 0)
             (size 1.6 1.2)
-            (layers "F.Cu" "F.Mask" "F.Paste")
-            (net 5 "VDD")
+            (layers "F.Cu" "F.Paste" "F.Mask")
+            (net 5 "VCC")
         )
         (pad "2" smd rect
             (at -2.35 1.65 0)
             (size 1.6 1.2)
-            (layers "F.Cu" "F.Mask" "F.Paste")
+            (layers "F.Cu" "F.Paste" "F.Mask")
             (net 2 "DOUT")
         )
@@
             (at 2.35 1.65 0)
             (size 1.6 1.2)
-            (layers "F.Cu" "F.Mask" "F.Paste")
-            (net 4 "gnd")
+            (layers "F.Cu" "F.Paste" "F.Mask")
+            (net 4 "GND")
         )
         (pad "4" smd rect
             (at 2.35 -1.65 0)
             (size 1.6 1.2)
-            (layers "F.Cu" "F.Mask" "F.Paste")
+            (layers "F.Cu" "F.Paste" "F.Mask")
             (net 1 "DIN")
         )
-        (embedded_fonts no)
         (model "${KIPRJMOD}/../../parts/Worldsemi_WS2812C/LED-SMD_4P-L5.0-W5.0-LS5.4-TL-1.step"
             (offset
@@
             )
         )
-        (property "__atopile_lib_fp_hash__" "0d4373b2-7efa-330f-4ab5-b88e00116aa8"
+        (property "__atopile_lib_fp_hash__" "26ec4086-6a41-2a44-f462-3459247aa05a"
             (at 0 0 0)
             (layer "User.9")
@@
             )
         )
-        (property "__atopile_lib_fp_hash__" "f09d99df-ed19-5d64-860b-d0dc74491bc0"
+        (property "__atopile_lib_fp_hash__" "f8a97365-7255-729e-24e5-6102db053d76"
             (at 0 0 0)
             (layer "User.9")
@@
             (size 0.79 0.54)
             (layers "F.Cu" "F.Paste" "F.Mask")
-            (net 4 "gnd")
+            (net 4 "GND")
         )
         (pad "1" smd rect
@@
             (size 0.79 0.54)
             (layers "F.Cu" "F.Paste" "F.Mask")
-            (net 5 "VDD")
+            (net 5 "VCC")
         )
         (model "${KIPRJMOD}/../../parts/Samsung_Electro_Mechanics_CL05B104KO5NNNC/C0402_L1.0-W0.5-H0.5.step"
