File: packages/worldsemi-ws2812c-5050/layouts/strip/strip.kicad_pcb (KiCad board)
At the start: 2 copper layers, 15 parts

Commit message: Rename pjrc-teensy_4_1 to pjrc-teensy-4-1
- Renamed package directory from pjrc-teensy_4_1 to pjrc-teensy-4-1
- Updated package naming convention to use hyphens instead of underscores
- Package marked as 'Done' in package-todos.md
- Fixed formatting issues (end-of-file and trailing whitespace)
Connections:
- net -DOUT-0 renamed data_out-DOUT
- net -DOUT-1 renamed leds[1]-data_in-DOUT
- net -DOUT-2 renamed leds[2]-data_in-DOUT
- net -DOUT-3 renamed leds[3]-data_in-DOUT
- net -DOUT-4 renamed leds[4]-data_in-DOUT
- net VDD renamed VCC
- net gnd renamed GND
- net leds[0]-DIN renamed data_protection_r-DIN-0
- net leds[1]-DIN renamed data_protection_r-DIN-1
- net leds[2]-DIN renamed data_protection_r-DIN-2
- net leds[3]-DIN renamed data_protection_r-DIN-3
- net leds[4]-DIN renamed data_protection_r-DIN-4
