File: packages/st-lis3dh/layouts/default/default.kicad_pcb (KiCad board)
At the start: 2 copper layers, 6 parts

Commit message: multipackage: Run builds with latest compiler to fix frozen errors (#183)
* fix rohm-bh1750

* fix rj45-connectors

* fix sensirion-scd40

* fix sensirion-scd41

* update package versions for release

* sensirion-sgp40: LLM Update with 0.12.4

Updated sensirion-sgp40 package to work with atopile compiler version 0.12.4.

Changes made:
- Updated requires-atopile from ^0.10.8 to ^0.12.4
- Updated package version from 0.1.0 to 0.1.1
- Rebuilt layouts with new compiler (net naming improvements)
- All builds pass: ato build, ato build --frozen, ato package verify -s

🤖 Generated with [Claude Code](https://claude.ai/code)

Co-Authored-By: Claude <noreply@anthropic.com>

* sensirion-sht31: LLM Update with 0.12.4

Updated sensirion-sht31 package to work with atopile compiler version 0.12.4.

Changes made:
- Updated requires-atopile from ^0.10.8 to ^0.12.4
- Updated package version from 0.1.0 to 0.1.1
- Rebuilt layouts with new compiler (net naming improvements)
- All builds pass: ato build, ato build --frozen, ato package verify -s

🤖 Generated with [Claude Code](https://claude.ai/code)

Co-Authored-By: Claude <noreply@anthropic.com>

* sensirion-sht40: LLM Update with 0.12.4

Updated sensirion-sht40 package to work with atopile compiler version 0.12.4.

Changes made:
- Updated requires-atopile from ^0.10.8 to ^0.12.4
- Updated package version from 0.1.0 to 0.1.1
- Rebuilt layouts with new compiler (net naming improvements)
- All builds pass: ato build, ato build --frozen, ato package verify -s

🤖 Generated with [Claude Code](https://claude.ai/code)

Co-Authored-By: Claude <noreply@anthropic.com>

* sensirion-sht41: LLM Update with 0.12.4

Updated sensirion-sht41 package to work with atopile compiler version 0.12.4.

Changes made:
- Updated requires-atopile from ^0.10.8 to ^0.12.4
- Updated package version from 0.1.0 to 0.1.1
- Rebuilt layouts with new compiler (net naming improvements)
- All builds pass: ato build, ato build --frozen, ato package verify -s

🤖 Generated wit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
Connections:
- net SCL_SPC renamed SCL
- net SDA_SDI_SDO renamed MOSI
- net SDO_SA0 renamed address_bit_0
- net VDD renamed power_core-VCC
- net gnd renamed GND
- net hv renamed power_io-VCC
- net package.footprint.pins[8].net-net renamed footprint-net-0
- net package.footprint.pins[9].net-net renamed footprint-net-1
