File: packages/st-lis3dh/layouts/default/default.kicad_pcb (KiCad board)
At the start: 2 copper layers, 6 parts

Commit message: st-lis3dh: package update to v0.2.0, ato:^0.14.0 (#337)
Build targets:
  default = rc0
  usage = rc0
Package Verify: rc0
Version: 0.1.2 -> 0.2.0
Requires ato: ^0.14.0
Parts:
- C1, C2: value 100nF ±10% 16V X7R -> 1±10.0%F
- R1, R2, R3: value 10kΩ ±1% 62.5mW -> 10000±1.0%Ω
Connections:
- net ADC1 renamed 16
- net ADC2 renamed 15
- net ADC3 renamed 13
- net INT1 renamed 11
- net INT2 renamed 9
- net power_core-VCC renamed decoupling_caps[0]-power-hv
- net power_io-VCC renamed hv
- C1 pad 2: GND -> lv
- C2 pad 2: GND -> lv
- U1 pad 12: GND -> lv
- U1 pad 2: footprint-net-0 -> (no net)
- U1 pad 3: footprint-net-1 -> (no net)
- U1 pad 5: GND -> lv
- U1 pad 7: address_bit_0 -> lv
Routing:
- net GND: track 6.25 -> 0.00 mm, vias 3 -> 0
- net 14: track 0.00 -> 6.25 mm, vias 0 -> 3
