File: packages/vishay-veml7700/layouts/default/default.kicad_pcb (KiCad board)
At the start: 2 copper layers, 4 parts

Commit message: multipackage: Run builds with latest compiler to fix frozen errors (#183)
* fix rohm-bh1750

* fix rj45-connectors

* fix sensirion-scd40

* fix sensirion-scd41

* update package versions for release

* sensirion-sgp40: LLM Update with 0.12.4

Updated sensirion-sgp40 package to work with atopile compiler version 0.12.4.

Changes made:
- Updated requires-atopile from ^0.10.8 to ^0.12.4
- Updated package version from 0.1.0 to 0.1.1
- Rebuilt layouts with new compiler (net naming improvements)
- All builds pass: ato build, ato build --frozen, ato package verify -s

🤖 Generated with [Claude Code](https://claude.ai/code)

Co-Authored-By: Claude <noreply@anthropic.com>

* sensirion-sht31: LLM Update with 0.12.4

Updated sensirion-sht31 package to work with atopile compiler version 0.12.4.

Changes made:
- Updated requires-atopile from ^0.10.8 to ^0.12.4
- Updated package version from 0.1.0 to 0.1.1
- Rebuilt layouts with new compiler (net naming improvements)
- All builds pass: ato build, ato build --frozen, ato package verify -s

🤖 Generated with [Claude Code](https://claude.ai/code)

Co-Authored-By: Claude <noreply@anthropic.com>

* sensirion-sht40: LLM Update with 0.12.4

Updated sensirion-sht40 package to work with atopile compiler version 0.12.4.

Changes made:
- Updated requires-atopile from ^0.10.8 to ^0.12.4
- Updated package version from 0.1.0 to 0.1.1
- Rebuilt layouts with new compiler (net naming improvements)
- All builds pass: ato build, ato build --frozen, ato package verify -s

🤖 Generated with [Claude Code](https://claude.ai/code)

Co-Authored-By: Claude <noreply@anthropic.com>

* sensirion-sht41: LLM Update with 0.12.4

Updated sensirion-sht41 package to work with atopile compiler version 0.12.4.

Changes made:
- Updated requires-atopile from ^0.10.8 to ^0.12.4
- Updated package version from 0.1.0 to 0.1.1
- Rebuilt layouts with new compiler (net naming improvements)
- All builds pass: ato build, ato build --frozen, ato package verify -s

🤖 Generated wit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
Connections:
- net VDD renamed VCC
- net gnd renamed GND
Changed lines of the file:
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@@
     )
     (net 0 "")
-    (net 1 "gnd")
+    (net 1 "GND")
     (net 2 "SCL")
-    (net 3 "VDD")
+    (net 3 "VCC")
     (net 4 "SDA")
     (footprint "Samsung_Electro_Mechanics_CL05B104KO5NNNC:C0402"
@@
             )
         )
-        (property "__atopile_lib_fp_hash__" "95674ebb-631f-c47a-aee5-cedff8134a1e"
+        (property "__atopile_lib_fp_hash__" "f8a97365-7255-729e-24e5-6102db053d76"
             (at 0 0 0)
             (layer "User.9")
@@
             (size 0.79 0.54)
             (layers "F.Cu" "F.Paste" "F.Mask")
-            (net 1 "gnd")
+            (net 1 "GND")
         )
         (pad "1" smd rect
@@
             (size 0.79 0.54)
             (layers "F.Cu" "F.Paste" "F.Mask")
-            (net 3 "VDD")
+            (net 3 "VCC")
         )
         (model "${KIPRJMOD}/../../parts/Samsung_Electro_Mechanics_CL05B104KO5NNNC/C0402_L1.0-W0.5-H0.5.step"
@@
             )
         )
-        (property "__atopile_lib_fp_hash__" "1a56f300-5712-5176-01d9-e086b76422ef"
+        (property "__atopile_lib_fp_hash__" "ac993d00-cd2e-9909-323a-aafc825a9032"
             (at 0 0 0)
             (layer "User.9")
@@
             (size 0.57 0.54)
             (layers "F.Cu" "F.Paste" "F.Mask")
-            (net 3 "VDD")
+            (net 3 "VCC")
         )
         (model "${KIPRJMOD}/../../parts/UNI_ROYAL_0402WGF1002TCE/R0402_L1.0-W0.5-H0.4.step"
@@
             (at 0 0 0)
             (layer "User.9")
-            (hide yes)
-            (effects
-                (font
-                    (size 0.125 0.125)
-                    (thickness 0.01875)
-                )
-            )
-        )
-        (property "__atopile_lib_fp_hash__" "2c9aa7eb-a53d-4c7e-01f7-59ff98661ca5"
+            (hide no)
+            (effects
+                (font
+                    (size 0.125 0.125)
+                    (thickness 0.01875)
+                )
+                (hide yes)
+            )
+        )
+        (property "__atopile_lib_fp_hash__" "02a6fe27-684e-3a60-ca5d-cf982d06e4ca"
             (at 0 0 0)
             (layer "User.9")
@@
         )
         (fp_line
+            (start -3.39 -1.84)
+            (end -2.86 -1.31)
+            (stroke
+                (width 0.25)
+                (type solid)
+            )
+            (layer "F.SilkS")
+        )
+        (fp_line
+            (start -2.86 -1.31)
+            (end 2.87 -1.31)
+            (stroke
+                (width 0.25)
+                (type solid)
+            )
+            (layer "F.SilkS")
+        )
+        (fp_line
+            (start 2.87 -1.31)
+            (end 3.4 -1.84)
+            (stroke
+                (width 0.25)
+                (type solid)
+            )
+            (layer "F.SilkS")
+        )
+        (fp_line
+            (start -2.53 0.5)
+            (end -3.4 0.5)
+            (stroke
+                (width 0.25)
+                (type solid)
+            )
+            (layer "F.SilkS")
+        )
+        (fp_line
+            (start -3.4 0.5)
+            (end -3.4 -1.84)
+            (stroke
+                (width 0.25)
+                (type solid)
+            )
+            (layer "F.SilkS")
+        )
+        (fp_line
             (start -3.4 -1.84)
             (end 3.4 -1.84)
@@
         )
         (fp_line
-            (start -3.4 0.5)
-            (end -3.4 -1.84)
+            (start 3.4 -1.84)
+            (end 3.4 0.5)
             (stroke
                 (width 0.25)
@@
         )
         (fp_line
-            (start -3.39 -1.84)
-            (end -2.86 -1.31)
-            (stroke
-                (width 0.25)
-                (type solid)
-            )
-            (layer "F.SilkS")
-        )
-        (fp_line
-            (start -2.86 -1.31)
-            (end 2.87 -1.31)
-            (stroke
-                (width 0.25)
-                (type solid)
-            )
-            (layer "F.SilkS")
-        )
-        (fp_line
-            (start -2.53 0.5)
-            (end -3.4 0.5)
+            (start 3.4 0.5)
+            (end 2.54 0.5)
             (stroke
                 (width 0.25)
@@
             (start 1.28 0.5)
             (end 1.27 0.5)
-            (stroke
-                (width 0.25)
-                (type solid)
-            )
-            (layer "F.SilkS")
-        )
-        (fp_line
-            (start 2.87 -1.31)
-            (end 3.4 -1.84)
-            (stroke
-                (width 0.25)
-                (type solid)
-            )
-            (layer "F.SilkS")
-        )
-        (fp_line
-            (start 3.4 -1.84)
-            (end 3.4 0.5)
-            (stroke
-                (width 0.25)
-                (type solid)
-            )
-            (layer "F.SilkS")
-        )
-        (fp_line
-            (start 3.4 0.5)
-            (end 2.54 0.5)
             (stroke
                 (width 0.25)
@@
             (layer "F.Fab")
         )
+        (fp_text user "%R"
+            (at 0 0 0)
+            (layer "F.Fab")
+            (effects
+                (font
+                    (size 1 1)
+                    (thickness 0.15)
+                )
+            )
+            (unlocked no)
+        )
         (fp_text user "${REFERENCE}"
             (at 0 -4 0)
             (layer "F.SilkS")
-            (hide yes)
-            (effects
-                (font
-                    (size 1 1)
-                    (thickness 0.15)
-                )
-                (hide yes)
-            )
-            (unlocked no)
-        )
-        (fp_text user "${REFERENCE}"
-            (at 0 0 0)
-            (layer "F.Fab")
             (effects
                 (font
@@
             (at 1.9 0 0)
             (size 0.8 1.8)
-            (layers "F.Cu" "F.Mask" "F.Paste")
+            (layers "F.Cu" "F.Paste" "F.Mask")
             (net 2 "SCL")
         )
@@
             (at 0.63 0 0)
             (size 0.8 1.8)
-            (layers "F.Cu" "F.Mask" "F.Paste")
-            (net 3 "VDD")
+            (layers "F.Cu" "F.Paste" "F.Mask")
+            (net 3 "VCC")
         )
         (pad "3" smd rect
             (at -0.63 0 0)
             (size 0.8 1.8)
-            (layers "F.Cu" "F.Mask" "F.Paste")
-            (net 1 "gnd")
+            (layers "F.Cu" "F.Paste" "F.Mask")
+            (net 1 "GND")
         )
         (pad "4" smd rect
             (at -1.91 0 0)
             (size 0.8 1.8)
-            (layers "F.Cu" "F.Mask" "F.Paste")
+            (layers "F.Cu" "F.Paste" "F.Mask")
             (net 4 "SDA")
         )
-        (embedded_fonts no)
         (model "${KIPRJMOD}/../../parts/VISHAY_VEML7700_TR/LED-SMD_4P-L6.8-W2.4_VEML7700-TR.STEP"
             (offset
@@
             )
         )
-        (property "__atopile_lib_fp_hash__" "1a56f300-5712-5176-01d9-e086b76422ef"
+        (property "__atopile_lib_fp_hash__" "ac993d00-cd2e-9909-323a-aafc825a9032"
             (at 0 0 0)
             (layer "User.9")
@@
             (size 0.57 0.54)
             (layers "F.Cu" "F.Paste" "F.Mask")
-            (net 3 "VDD")
+            (net 3 "VCC")
         )
         (model "${KIPRJMOD}/../../parts/UNI_ROYAL_0402WGF1002TCE/R0402_L1.0-W0.5-H0.4.step"
