File: packages/vishay-veml7700/layouts/default/default.kicad_pcb (KiCad board)
At the start: 2 copper layers, 4 parts

Commit message: many packages building
Parts:
- C1: value 100nF ±10% 16V X7R -> 1.0000000000000001e-07F
- R1, R2: value 10kΩ ±1% 62.5mW -> 10000.0Ω
Connections:
- net GND renamed lv
- net VCC renamed hv

Commit message: update parts
Parts:
- C1: value 1.0000000000000001e-07F -> 1±20.0%F
- R1, R2: value 10000.0Ω -> 10000±5.0%Ω
Changed lines of the file:
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@@
 			(usegerberadvancedattributes yes)
 			(creategerberjobfile yes)
-			(dashed_line_dash_ratio 12.000000)
-			(dashed_line_gap_ratio 3.000000)
+			(dashed_line_dash_ratio 12)
+			(dashed_line_gap_ratio 3)
 			(svgprecision 4)
 			(plotframeref no)
@@
 			(hpglpennumber 1)
 			(hpglpenspeed 20)
-			(hpglpendiameter 15.000000)
+			(hpglpendiameter 15)
 			(pdf_front_fp_property_popups yes)
 			(pdf_back_fp_property_popups yes)
@@
 			)
 		)
-		(property "Value" "1.0000000000000001e-07F"
+		(property "Value" "1±20.0%F"
 			(at 0 4 180)
 			(layer "F.Fab")
@@
 			)
 		)
-		(property "capacitance" "1.0000000000000001e-07±10.0%F"
-			(at 0 0 0)
-			(layer "User.9")
-			(hide yes)
-		)
-		(property "max_voltage" "16.0V"
+		(property "capacitance" "1±20.0%F"
+			(at 0 0 0)
+			(layer "User.9")
+			(hide yes)
+		)
+		(property "max_voltage" "{ℝ+}V"
 			(at 0 0 0)
 			(layer "User.9")
@@
 			)
 		)
-		(property "Value" "10000.0Ω"
+		(property "Value" "10000±5.0%Ω"
 			(at 0 4)
 			(layer "F.Fab")
@@
 			)
 		)
-		(property "resistance" "10000.0±1.0%Ω"
-			(at 0 0 0)
-			(layer "User.9")
-			(hide yes)
-		)
-		(property "max_power" "0.0625W"
-			(at 0 0 0)
-			(layer "User.9")
-			(hide yes)
-		)
-		(property "max_voltage" "50.0V"
+		(property "resistance" "10000±5.0%Ω"
+			(at 0 0 0)
+			(layer "User.9")
+			(hide yes)
+		)
+		(property "max_power" "{ℝ+}W"
+			(at 0 0 0)
+			(layer "User.9")
+			(hide yes)
+		)
+		(property "max_voltage" "{ℝ+}V"
 			(at 0 0 0)
 			(layer "User.9")
@@
 			)
 		)
-		(property "Value" "10000.0Ω"
+		(property "Value" "10000±5.0%Ω"
 			(at 0 4)
 			(layer "F.Fab")
@@
 			)
 		)
-		(property "resistance" "10000.0±1.0%Ω"
-			(at 0 0 0)
-			(layer "User.9")
-			(hide yes)
-		)
-		(property "max_power" "0.0625W"
-			(at 0 0 0)
-			(layer "User.9")
-			(hide yes)
-		)
-		(property "max_voltage" "50.0V"
-			(at 0 0 0)
-			(layer "User.9")
+		(property "resistance" "10000±5.0%Ω"
+			(at 0 0 0)
+			(layer "User.9")
+			(hide yes)
+		)
+		(property "max_power" "{ℝ+}W"
+			(at 0 0 0)
+			(layer "User.9")
+			(hide yes)
+		)
+		(property "max_voltage" "{ℝ+}V"
+			(at 0 0 0)
+			(layer "User.9")
