File: packages/ti-pcm1789/layouts/default/default.kicad_pcb (KiCad board)
At the start: 2 copper layers, 17 parts

Commit message: pcb tidy up
Parts:
- moved R9 181.9 mm to (148.9, 94.5), turned to 90 degrees
- moved R8 175.5 mm to (147.9, 94.5), turned to 90 degrees
Routing:
- net power_3v3-VCC: track 0.00 -> 18.1 mm, vias 0 -> 3
- net (no net): track 15.9 -> 0.00 mm, vias 2 -> 0
- net SCL: track 0.00 -> 2.79 mm
- net SDA: track 0.00 -> 2.75 mm

Commit message: update parts
Parts:
- C1, C2, C3: value 1µF ±10% 25V X5R -> 1e-06±10.0%F
- C4, C5, C6, C7: value 10µF ±10% 10V X5R -> 9.999±10.0%F
- R1: value 10kΩ ±1% 62.5mW -> 10000±2.0%Ω
- R2, R3, R4, R5: value 22Ω ±1% 62.5mW -> 22±2.0%Ω
- R6, R7, R8, R9: value 10kΩ ±1% 62.5mW -> 10000±5.0%Ω
Connections:
- net ZERO1 renamed 19
- net _power_vcom-VCC renamed hv
- net power_3v3-VCC renamed decoupling_1uf[0]-power-hv
- net power_5v-VCC renamed decoupling_1uf[2]-power-hv
- C1 pad 2: GND -> lv
- C2 pad 2: GND -> lv
- C3 pad 2: GND -> lv
- C4 pad 2: GND -> lv
- C5 pad 2: GND -> lv
- C6 pad 2: GND -> lv
- C7 pad 2: GND -> lv
- U1 pad 10: GND -> lv
- U1 pad 15: GND -> lv
- U1 pad 20: GND -> lv
- U1 pad 23: address_bit_0 -> lv
- U1 pad 24: address_bit_1 -> lv
- U1 pad 7: GND -> lv
Routing:
- net lv: track 0.00 -> 25.7 mm, vias 0 -> 5
- net GND: track 25.7 -> 0.00 mm, vias 5 -> 0
