File: packages/worldsemi-ws2812b/layouts/default/default.kicad_pcb (KiCad board)
At the start: 2 copper layers, 2 parts

Commit message: review tool updates
Parts:
- C1: value 100nF ±10% 16V X7R -> 1.0000000000000001e-07F
Connections:
- net GND renamed lv
- net VCC renamed hv

Commit message: update parts
Parts:
- C1: value 1.0000000000000001e-07F -> 1±20.0%F
Changed lines of the file:
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@@
 			(usegerberadvancedattributes yes)
 			(creategerberjobfile yes)
-			(dashed_line_dash_ratio 12.000000)
-			(dashed_line_gap_ratio 3.000000)
+			(dashed_line_dash_ratio 12)
+			(dashed_line_gap_ratio 3)
 			(svgprecision 4)
 			(plotframeref no)
@@
 			(hpglpennumber 1)
 			(hpglpenspeed 20)
-			(hpglpendiameter 15.000000)
+			(hpglpendiameter 15)
 			(pdf_front_fp_property_popups yes)
 			(pdf_back_fp_property_popups yes)
@@
 			)
 		)
-		(property "Value" "1.0000000000000001e-07F"
+		(property "Value" "1±20.0%F"
 			(at 0 4 180)
 			(layer "F.Fab")
@@
 			)
 		)
-		(property "capacitance" "1.0000000000000001e-07±10.0%F"
+		(property "capacitance" "1±20.0%F"
 			(at 0 0 0)
 			(layer "User.9")
 			(hide yes)
 		)
-		(property "max_voltage" "16.0V"
+		(property "max_voltage" "{ℝ+}V"
 			(at 0 0 0)
 			(layer "User.9")
