File: packages/ylptech-byyxx/layouts/B1205S/B1205S.kicad_pcb (KiCad board)
At the start: 2 copper layers, 3 parts

Commit message: ylptech-byyxx: sync build outputs
Build targets:
  B0505S = rc0
  B1205S = rc0
  usage = rc0
Package Verify: rc0
Parts:
- C1: value 2.2e-06F -> [capacitance: unknown]
- C2: value 9.999999999999999e-06F -> [capacitance: unknown]
Changed lines of the file:
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@@
 			)
 		)
-		(property "Value" "9.999999999999999e-06F"
+		(property "Value" "[capacitance: unknown]"
 			(at 0 4 270)
 			(layer "F.Fab")
@@
 			)
 		)
-		(property "capacitance" "9.999999999999999e-06±10.0%F"
-			(at 0 0 0)
-			(layer "User.9")
-			(hide yes)
-		)
-		(property "max_voltage" "25.0V"
-			(at 0 0 0)
-			(layer "User.9")
-			(hide yes)
-		)
-		(property "temperature_coefficient" "X5R"
+		(property "capacitance" "[capacitance: unknown]"
+			(at 0 0 0)
+			(layer "User.9")
+			(hide yes)
+		)
+		(property "max_voltage" "[max_voltage: unknown]"
+			(at 0 0 0)
+			(layer "User.9")
+			(hide yes)
+		)
+		(property "temperature_coefficient" "[temperature_coefficient: unknown]"
 			(at 0 0 0)
 			(layer "User.9")
@@
 			)
 		)
-		(property "Value" "2.2e-06F"
+		(property "Value" "[capacitance: unknown]"
 			(at 0 4 270)
 			(layer "F.Fab")
@@
 			)
 		)
-		(property "capacitance" "2.2e-06±10.0%F"
-			(at 0 0 0)
-			(layer "User.9")
-			(hide yes)
-		)
-		(property "max_voltage" "25.0V"
-			(at 0 0 0)
-			(layer "User.9")
-			(hide yes)
-		)
-		(property "temperature_coefficient" "X7R"
-			(at 0 0 0)
-			(layer "User.9")
+		(property "capacitance" "[capacitance: unknown]"
+			(at 0 0 0)
+			(layer "User.9")
+			(hide yes)
+		)
+		(property "max_voltage" "[max_voltage: unknown]"
+			(at 0 0 0)
+			(layer "User.9")
+			(hide yes)
+		)
+		(property "temperature_coefficient" "[temperature_coefficient: unknown]"
+			(at 0 0 0)
+			(layer "User.9")
