File: packages/worldsemi-ws2812c/layouts/matrix/matrix.kicad_pcb (KiCad board)
At the start: 2 copper layers, 75 parts

Commit message: worldsemi-ws2812c: update for ^0.14.0 (#230)
* worldsemi-ws2812c: package update [reviewer:Narayan Powderly] [ato:^0.14.0]

Builds: default=rc0, matrix=rc0, strip=rc0, usage=rc0, ws2812c-2020=rc0, ws2812c-4020=rc0, ws2812c-5050=rc0
Verify: rc0
Version: 0.2.1 -> 0.3.0

* Update main.yml from main

Syncs GitHub Actions workflow configuration.

* ci: update workflow from main (fix package publish git issue)

* worldsemi-ws2812c: sync build outputs

Build targets:
  matrix = rc0
  strip = rc0
  usage = rc0
  ws2812c-2020 = rc0
  ws2812c-4020 = rc0
  ws2812c-5050 = rc0
Package Verify: rc0

---------

Co-authored-by: Nicholas Krstevski <nick@atopile.io>
Co-authored-by: Nick Krstevski <51719418+nickkrstevski@users.noreply.github.com>
Parts:
- C13, C14, C15, C16, C17, C2, C24, C25, C26, C27, C28, C3, C35, C36, C37, C38, C39, C4, C46, C47, C48, C49, C5, C50, C6: value 100nF ±10% 16V X7R -> [capacitance: unknown]
- R1, R11, R12, R13, R14, R15, R2, R21, R22, R23, R24, R25, R3, R31, R32, R33, R34, R35, R4, R41, R42, R43, R44, R45, R5: value 330Ω ±1% 62.5mW -> [resistance: unknown]
Connections:
- net GND renamed lv
- net VCC renamed hv
- net data_protection_r-DIN-0 renamed DIN
- net data_protection_r-DIN-1 renamed strips[0].leds[1]-DIN
- net data_protection_r-DIN-10 renamed strips[2].leds[0]-DIN
- net data_protection_r-DIN-11 renamed strips[2].leds[1]-DIN
- net data_protection_r-DIN-12 renamed strips[2].leds[2]-DIN
- net data_protection_r-DIN-13 renamed strips[2].leds[3]-DIN
- net data_protection_r-DIN-14 renamed strips[2].leds[4]-DIN
- net data_protection_r-DIN-15 renamed strips[3].leds[0]-DIN
- net data_protection_r-DIN-16 renamed strips[3].leds[1]-DIN
- net data_protection_r-DIN-17 renamed strips[3].leds[2]-DIN
- net data_protection_r-DIN-18 renamed strips[3].leds[3]-DIN
- net data_protection_r-DIN-19 renamed strips[3].leds[4]-DIN
- net data_protection_r-DIN-2 renamed strips[0].leds[2]-DIN
- net data_protection_r-DIN-20 renamed strips[4].leds[0]-DIN
- net data_protection_r-DIN-21 renamed strips[4].leds[1]-DIN
- net data_protection_r-DIN-22 renamed strips[4].leds[2]-DIN
- net data_protection_r-DIN-23 renamed strips[4].leds[3]-DIN
- net data_protection_r-DIN-24 renamed strips[4].leds[4]-DIN
- net data_protection_r-DIN-3 renamed strips[0].leds[3]-DIN
- net data_protection_r-DIN-4 renamed strips[0].leds[4]-DIN
- net data_protection_r-DIN-5 renamed strips[1].leds[0]-DIN
- net data_protection_r-DIN-6 renamed strips[1].leds[1]-DIN
- net data_protection_r-DIN-7 renamed strips[1].leds[2]-DIN
- net data_protection_r-DIN-8 renamed strips[1].leds[3]-DIN
- net data_protection_r-DIN-9 renamed strips[1].leds[4]-DIN
- net leds[1]-data_in-DOUT-0 renamed DOUT
- net leds[2]-data_in-DOUT-0 renamed leds[2]-data_in-DOUT
- net leds[3]-data_in-DOUT-0 renamed leds[3]-data_in-DOUT
- net leds[4]-data_in-DOUT-0 renamed leds[4]-data_in-DOUT
- net strips[0]-data_in-line renamed line
- LED11 pad 2: leds[1]-data_in-DOUT-1 -> leds[1]-data_in-DOUT
- LED21 pad 2: leds[1]-data_in-DOUT-2 -> leds[1]-data_in-DOUT-1
- LED31 pad 2: leds[1]-data_in-DOUT-3 -> leds[1]-data_in-DOUT-2
- LED41 pad 2: leds[1]-data_in-DOUT-4 -> leds[1]-data_in-DOUT-3
- R12 pad 1: leds[1]-data_in-DOUT-1 -> leds[1]-data_in-DOUT
- R22 pad 1: leds[1]-data_in-DOUT-2 -> leds[1]-data_in-DOUT-1
- R32 pad 1: leds[1]-data_in-DOUT-3 -> leds[1]-data_in-DOUT-2
- R42 pad 1: leds[1]-data_in-DOUT-4 -> leds[1]-data_in-DOUT-3
Routing:
- net leds[1]-data_in-DOUT-4: track 1.75 -> 0.00 mm
- net leds[1]-data_in-DOUT: track 0.00 -> 1.75 mm

Commit message: worldsemi-ws2812c: package update version 0.3.0, ato 0.14.0, frozen fix (#359)
* worldsemi-ws2812c: package update [reviewer:Narayan Powderly] [ato:^0.14.0]

Builds: default=rc0, matrix=rc0, strip=rc0, usage=rc0, ws2812c-2020=rc0, ws2812c-4020=rc0, ws2812c-5050=rc0
Verify: rc0
Version: 0.2.1 -> 0.3.0

* Update main.yml from main

Syncs GitHub Actions workflow configuration.

* ci: update workflow from main (fix package publish git issue)

* manual fix package

---------

Co-authored-by: Narayan Powderly <narayan@atopile.io>
Co-authored-by: Narayan Powderly <napowderly@gmail.com>
Parts:
- C13, C14, C15, C16, C17, C2, C24, C25, C26, C27, C28, C3, C35, C36, C37, C38, C39, C4, C46, C47, C48, C49, C5, C50, C6: value [capacitance: unknown] -> 1F
- R1, R11, R12, R13, R14, R15, R2, R21, R22, R23, R24, R25, R3, R31, R32, R33, R34, R35, R4, R41, R42, R43, R44, R45, R5: value [resistance: unknown] -> 330Ω
