File: packages/worldsemi-ws2812c/layouts/matrix/matrix.kicad_pcb (KiCad board)
At the start: 2 copper layers, 75 parts

Commit message: Widen voltage range on all addressable RGB LED packages to 3V-5.5V (#450)
* Widen voltage range on all addressable RGB LED packages to 3V-5.5V

Real-world testing shows WS2812B/SK6805 LEDs operate reliably down
to ~3V (blue channel dims first). Update voltage assertions from
their conservative datasheet values to match practical usage,
enabling direct 3.3V and LiPo battery operation.

Updated packages:
- opsco-sk6805-ec15: 0.3.0 → 0.4.0
- opsco-sk6805-ec20: 0.4.1 → 0.5.0
- opsco-sk6805-side: 0.5.0 → 0.6.0
- worldsemi-ws2812b: 0.3.0 → 0.4.0
- worldsemi-ws2812c: 0.3.0 → 0.4.0

Co-Authored-By: Claude Opus 4.6 (1M context) <noreply@anthropic.com>

* Rebuild layouts for all addressable RGB LED packages

Co-Authored-By: Claude Opus 4.6 (1M context) <noreply@anthropic.com>

* worldsemi-ws2812b: Remove unused Resistor import

Co-Authored-By: Claude Opus 4.6 (1M context) <noreply@anthropic.com>

---------

Co-authored-by: Claude Opus 4.6 (1M context) <noreply@anthropic.com>
Parts:
- C13, C14, C15, C16, C17, C2, C24, C25, C26, C27, C28, C3, C35, C36, C37, C38, C39, C4, C46, C47, C48, C49, C5, C50, C6: value 1F -> 100nF ±10%
- R1, R11, R12, R13, R14, R15, R2, R21, R22, R23, R24, R25, R3, R31, R32, R33, R34, R35, R4, R41, R42, R43, R44, R45, R5: value 330Ω -> 330Ω ±1%; footprint YAGEO_RC0402FR_07330RL:R0402 -> UNI_ROYAL_0402WGF3300TCE:R0402
