File: packages/programming-headers/layouts/usage/usage.kicad_pcb (KiCad board)
At the start: 2 copper layers, 5 parts

Commit message: ready to rip
Parts:
- removed J1: , Tag-Connect_TC2050-IDC-NL_2x05_P1.27mm_Vertical:Tag-Connect_TC2050-IDC-NL_2x05_P1.27mm_Vertical
- moved CN2 142.2 mm to (52.2, 21.6)
- moved J2 132.5 mm to (37.4, 35.5), turned to -90 degrees
- moved CN1 101.5 mm to (59.0, 35.3)
- moved U1 97.8 mm to (44.4, 34.9)
Connections:
- net connector-net-1 renamed net
- net tc2050_arm_cortex-swd-N_RESET renamed swd-N_RESET

Commit message: update to 0.14.0
Connections:
- net _17 renamed 17
- net _19 renamed 19
- net _2 renamed 2
- net connector-_7-0 renamed 7
- net connector-_7-1 renamed idc_2_54mm_10pin_arm_cortex.connector-7
- net hdr_2_54mm_10pin_arm_cortex-jtag-TDI renamed TDI
- net hdr_2_54mm_10pin_arm_cortex-swd-N_TRST renamed N_TRST
- net hdr_2_54mm_10pin_arm_cortex-swd-TCK renamed CLK
- net hdr_2_54mm_10pin_arm_cortex-swd-TDO renamed SWO
- net hdr_2_54mm_10pin_arm_cortex-swd-TMS renamed DIO
- net hdr_2_54mm_10pin_arm_cortex-swd-VTREF-0 renamed hv
- net hdr_2_54mm_10pin_arm_cortex-swd-VTREF-1 renamed lv
- net idc_2_54mm_10pin_arm_cortex-swd-TCK renamed idc_2_54mm_10pin_arm_cortex-swd-CLK
- net idc_2_54mm_10pin_arm_cortex-swd-TDO renamed idc_2_54mm_10pin_arm_cortex-swd-SWO
- net idc_2_54mm_10pin_arm_cortex-swd-TMS renamed idc_2_54mm_10pin_arm_cortex-swd-DIO
- net idc_2_54mm_10pin_arm_cortex-swd-VTREF-0 renamed idc_2_54mm_10pin_arm_cortex-swd-hv
- net idc_2_54mm_10pin_arm_cortex-swd-VTREF-1 renamed idc_2_54mm_10pin_arm_cortex-swd-lv
- net idc_2_54mm_20pin_arm-jtag-RTCK renamed RTCK
- net idc_2_54mm_20pin_arm-jtag-VTREF-0 renamed jtag-hv
- net idc_2_54mm_20pin_arm-jtag-VTREF-1 renamed jtag-lv
- net jtag-N_RESET renamed N_RESET
- net jtag-TCK renamed TCK
- net jtag-TDO renamed TDO
- net jtag-TMS renamed TMS
- net tc2050_arm_cortex-swd-TCK renamed tc2050_arm_cortex-swd-CLK
- net tc2050_arm_cortex-swd-TDO renamed tc2050_arm_cortex-swd-SWO
- net tc2050_arm_cortex-swd-TMS renamed tc2050_arm_cortex-swd-DIO
- net tc2050_arm_cortex-swd-VTREF-0 renamed tc2050_arm_cortex-swd-hv
- net tc2050_arm_cortex-swd-VTREF-1 renamed tc2050_arm_cortex-swd-lv
- J2 pad : net -> (no net)
