File: packages/relays/layouts/LogicLevelRelaySPDT1A24V/LogicLevelRelaySPDT1A24V.kicad_pcb (KiCad board)
At the start: 2 copper layers, 6 parts

Commit message: fix relays build
Parts:
- R1, R2, R3: value 10kΩ ±1% 62.5mW -> 10kΩ
Connections:
- net GND renamed lv
- net drain renamed output

Commit message: add bistable relays + driver, fix coil and rest of the build
Connections:
- net output renamed contacts[1]
Changed lines of the file:
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@@
 	(net 5 "common")
 	(net 6 "cathode")
-	(net 7 "output")
+	(net 7 "contacts[1]")
 	(net 8 "lv")
 	(net 9 "anode")
@@
 			(size 1.25 0.7)
 			(layers "F.Cu" "F.Paste" "F.Mask")
-			(net 7 "output")
+			(net 7 "contacts[1]")
 		)
 		(model "${KIPRJMOD}/../../parts/Alpha___Omega_Semicon_AO3400A/SOT-23-3P_L2.9-W1.3-H1.0-LS2.4-P0.95.step"
@@
 			(drill 1.199896)
 			(layers "*.Cu" "*.Mask")
-			(net 7 "output")
+			(net 7 "contacts[1]")
 		)
 		(pad "10" thru_hole circle

Commit message: fix package check and build errors
Parts:
- R1, R2: value 10kΩ -> 10000Ω
- R3: value 10kΩ -> 47000Ω; footprint UNI_ROYAL_0402WGF1002TCE:R0402 -> UNI_ROYAL_0402WGF4702TCE:R0402
Changed lines of the file:
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@@
 	)
 	(setup
+		(stackup
+			(layer "F.SilkS"
+				(type "Top Silk Screen")
+			)
+			(layer "F.Paste"
+				(type "Top Solder Paste")
+			)
+			(layer "F.Mask"
+				(type "Top Solder Mask")
+				(color "Black")
+				(thickness 0.01)
+				(material "Solder mask")
+				(epsilon_r 3.3)
+			)
+			(layer "F.Cu"
+				(type "copper")
+				(thickness 0.035)
+			)
+			(layer "dielectric 1"
+				(type "core")
+				(thickness 1.51)
+				(material "FR4")
+				(epsilon_r 4.5)
+				(loss_tangent 0.02)
+			)
+			(layer "B.Cu"
+				(type "copper")
+				(thickness 0.035)
+			)
+			(layer "B.Mask"
+				(type "Bottom Solder Mask")
+				(color "Black")
+				(thickness 0.01)
+				(material "Solder mask")
+				(epsilon_r 3.3)
+			)
+			(layer "B.Paste"
+				(type "Bottom Solder Paste")
+			)
+			(layer "B.SilkS"
+				(type "Bottom Silk Screen")
+			)
+			(copper_finish "ENIG")
+		)
 		(pad_to_mask_clearance 0)
 		(allow_soldermask_bridges_in_footprints no)
@@
 	(net 8 "lv")
 	(net 9 "anode")
-	(footprint "UNI_ROYAL_0402WGF1002TCE:R0402"
+	(footprint "UNI_ROYAL_0402WGF4702TCE:R0402"
 		(layer "F.Cu")
 		(at 31.418854 2.401029 90)
@@
 			)
 		)
-		(property "Value" "10kΩ"
+		(property "Value" "47000Ω"
 			(at 0 4 90)
 			(layer "F.Fab")
@@
 			)
 		)
-		(property "Datasheet" "https://www.lcsc.com/datasheet/lcsc_datasheet_2411221126_UNI-ROYAL-Uniroyal-Elec-0402WGF1002TCE_C25744.pdf"
+		(property "Datasheet" "https://www.lcsc.com/datasheet/lcsc_datasheet_2206010100_UNI-ROYAL-Uniroyal-Elec-0402WGF4702TCE_C25792.pdf"
 			(at 0 0 90)
 			(layer "User.9")
@@
 			)
 		)
-		(property "LCSC" "C25744"
+		(property "LCSC" "C25792"
 			(at 0 0 90)
 			(layer "User.9")
@@
 			)
 		)
-		(property "Partnumber" "0402WGF1002TCE"
+		(property "Partnumber" "0402WGF4702TCE"
 			(at 0 0 90)
 			(layer "User.9")
@@
 			)
 		)
-		(property "PARAM_resistance" "{\"type\": \"Quantity_Interval_Disjoint\", \"data\": {\"intervals\": {\"type\": \"Numeric_Interval_Disjoint\", \"data\": {\"intervals\": [{\"type\": \"Numeric_Interval\", \"data\": {\"min\": 9900.000002235174, \"max\": 10099.999997764826}}]}}, \"unit\": \"ohm\"}}"
+		(property "PARAM_resistance" "{\"type\": \"Quantity_Interval_Disjoint\", \"data\": {\"intervals\": {\"type\": \"Numeric_Interval_Disjoint\", \"data\": {\"intervals\": [{\"type\": \"Numeric_Interval\", \"data\": {\"min\": 46530.00001050532, \"max\": 47469.99998949468}}]}}, \"unit\": \"ohm\"}}"
 			(at 0 0 90)
 			(layer "User.9")
@@
 			)
 		)
-		(property "resistance" "10±1.0%kΩ"
-			(at 0 0 0)
-			(layer "User.9")
-			(hide yes)
-		)
-		(property "max_power" "62.5mW"
+		(property "resistance" "47000±1.0%Ω"
+			(at 0 0 0)
+			(layer "User.9")
+			(hide yes)
+		)
+		(property "max_power" "0.062W"
 			(at 0 0 0)
 			(layer "User.9")
@@
 			(hide yes)
 		)
-		(property "lcsc_id" "C25744"
+		(property "lcsc_id" "C25792"
 			(at 0 0 0)
 			(layer "User.9")
@@
 		)
 		(embedded_fonts no)
-		(model "${KIPRJMOD}/../../parts/UNI_ROYAL_0402WGF1002TCE/R0402_L1.0-W0.5-H0.4.step"
+		(model "${KIPRJMOD}/../../parts/UNI_ROYAL_0402WGF4702TCE/R0402_L1.0-W0.5-H0.4.step"
 			(offset
 				(xyz 0 0 -0)
@@
 			)
 		)
-		(property "Value" "10kΩ"
+		(property "Value" "10000Ω"
 			(at 0 4 270)
 			(layer "F.Fab")
@@
 			)
 		)
-		(property "resistance" "10±1.0%kΩ"
-			(at 0 0 0)
-			(layer "User.9")
-			(hide yes)
-		)
-		(property "max_power" "62.5mW"
+		(property "resistance" "10000±1.0%Ω"
+			(at 0 0 0)
+			(layer "User.9")
+			(hide yes)
+		)
+		(property "max_power" "0.062W"
 			(at 0 0 0)
 			(layer "User.9")
@@
 			)
 		)
-		(property "Value" "10kΩ"
+		(property "Value" "10000Ω"
 			(at 0 4 270)
 			(layer "F.Fab")
@@
 			)
 		)
-		(property "resistance" "10±1.0%kΩ"
-			(at 0 0 0)
-			(layer "User.9")
-			(hide yes)
-		)
-		(property "max_power" "62.5mW"
-			(at 0 0 0)
-			(layer "User.9")
+		(property "resistance" "10000±1.0%Ω"
+			(at 0 0 0)
+			(layer "User.9")
+			(hide yes)
+		)
+		(property "max_power" "0.062W"
+			(at 0 0 0)
+			(layer "User.9")
