File: packages/ti-tps63020/layouts/usage/usage.kicad_pcb (KiCad board)
At the start: 2 copper layers, 12 parts

Commit message: Update 8 voltage divider packages for new ResistorVoltageDivider API (#447)
* Update 8 voltage divider packages for new ResistorVoltageDivider API

Migrate all packages using voltage dividers to the new API introduced
in atopile 0.14.x with the discrete sampling solver. Bump versions
(minor) and set requires-atopile to ^0.14.0.

Co-Authored-By: Claude Opus 4.6 (1M context) <noreply@anthropic.com>

* Update picked parts and layouts for new voltage divider values

Generated by `ato build` after updating voltage divider API.

Co-Authored-By: Claude Opus 4.6 (1M context) <noreply@anthropic.com>

* Restore feedback divider resistor positions from pre-rename layouts

Copy the (at X Y angle) coordinates from the old r_top/r_bottom
footprints to the new chain.resistors[0]/chain.resistors[1] footprints
so board layouts are preserved.

Co-Authored-By: Claude Opus 4.6 (1M context) <noreply@anthropic.com>

* Place tps63020 usage feedback divider resistors near IC

The chain.resistors[0/1] footprints were at origin (0,0). Placed
them adjacent to the converter package at (157, 103-104).

Co-Authored-By: Claude Opus 4.6 (1M context) <noreply@anthropic.com>

* Fix feedback divider resistor package to R0402 and place tps63020 resistors

- st-ldk220, ti-tlv75901, ti-tps82130: "0402" -> "R0402" for divider resistors
- ti-tps82130: rebuild picked parts with R0402 footprint
- ti-tps63020/default: place divider resistors near IC

Co-Authored-By: Claude Opus 4.6 (1M context) <noreply@anthropic.com>

* Remove #pragma experiment directives from all package .ato files

These features (TRAITS, FOR_LOOP, BRIDGE_CONNECT, MODULE_TEMPLATING)
are now first-class ato v1 language features and no longer require
pragma gates.

Co-Authored-By: Claude Opus 4.6 (1M context) <noreply@anthropic.com>

* Update CI to use latest tagged atopile release instead of main

Changes docker-tag from "main" to "latest" so builds use the latest
stable release (currently 0.15.0) rather than unreleased main branch code.
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
Parts:
- C1, C2: value 0F -> 10µF ±10%
- C3, C4, C5, C6: value 0F -> 22µF ±20%
- C7: value 0F -> 100nF ±10%
- L1: value L 0H -> L 1µH ±20%
- R1: value 150000Ω -> 107kΩ ±1%; footprint FOJAN_FRC0402F1503TS:R0402 -> UNI_ROYAL_0402WGF1073TCE:R0402
- R2: value 22000Ω -> 19.1kΩ ±1%; footprint UNI_ROYAL_0402WGF2202TCE:R0402 -> FOJAN_FRC0402F1912TS:R0402
- R3: value 1000000Ω -> 1MΩ ±1%
- moved R1 194.2 mm to (152.4, 110.2), turned to 270 degrees
- moved R2 186.8 mm to (151.9, 108.6), turned to 180 degrees
