File: packages/espressif-esp32-s3/layouts/usage/usage.kicad_pcb (KiCad board)
At the start: 2 copper layers, 8 parts

Commit message: espressif-esp32-s3, st-stm32h723: Fix cross-type bus parameter resolution (#451)
* espressif-esp32-s3, st-stm32h723: Fix cross-type bus parameter resolution

Same fix as espressif-esp32-c3 (#448): connect GPIO (ElectricLogic) to
ADC/USB/touch (ElectricSignal) at the .line level to avoid forming a
cross-type bus that breaks characteristic_impedance resolution.

ESP32-S3: fix USB d.p/d.n, touch[1-14], adc[1-20] connections
STM32H723: fix USB d.p/d.n connections

- espressif-esp32-s3: 0.2.1 → 0.3.0
- st-stm32h723: 0.1.2 → 0.2.0

Co-Authored-By: Claude Opus 4.6 (1M context) <noreply@anthropic.com>

* rebuild locally

* st-stm32h723: Remove unused imports and commented-out lan8742a ref

Co-Authored-By: Claude Opus 4.6 (1M context) <noreply@anthropic.com>

* st-stm32h723: Sync README usage block with usage.ato

Co-Authored-By: Claude Opus 4.6 (1M context) <noreply@anthropic.com>

---------

Co-authored-by: Claude Opus 4.6 (1M context) <noreply@anthropic.com>
Parts:
- C1: value 9.999F -> 10µF ±10%
- C2: value 1F -> 100nF ±10%
- C3: value 1e-06F -> 1µF ±10%
- R1, R2: value 10000Ω -> 10kΩ ±1%
Changed lines of the file:
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@@
 	)
 	(setup
+		(stackup
+			(layer "F.SilkS"
+				(type "Top Silk Screen")
+			)
+			(layer "F.Paste"
+				(type "Top Solder Paste")
+			)
+			(layer "F.Mask"
+				(type "Top Solder Mask")
+				(color "Black")
+				(thickness 0.01)
+				(material "Solder mask")
+				(epsilon_r 3.3)
+			)
+			(layer "F.Cu"
+				(type "copper")
+				(thickness 0.035)
+			)
+			(layer "dielectric 1"
+				(type "core")
+				(thickness 1.51)
+				(material "FR4")
+				(epsilon_r 4.5)
+				(loss_tangent 0.02)
+			)
+			(layer "B.Cu"
+				(type "copper")
+				(thickness 0.035)
+			)
+			(layer "B.Mask"
+				(type "Bottom Solder Mask")
+				(color "Black")
+				(thickness 0.01)
+				(material "Solder mask")
+				(epsilon_r 3.3)
+			)
+			(layer "B.Paste"
+				(type "Bottom Solder Paste")
+			)
+			(layer "B.SilkS"
+				(type "Bottom Silk Screen")
+			)
+			(copper_finish "ENIG")
+		)
 		(pad_to_mask_clearance 0)
 		(allow_soldermask_bridges_in_footprints no)
@@
 			)
 		)
-		(property "atopile_subaddresses" "[layouts/default/default.kicad_pcb:reset_switch.package]"
+		(property "atopile_subaddresses" "[.ato/modules/atopile/buttons/layouts/VerticalButton/VerticalButton.kicad_pcb:package, layouts/default/default.kicad_pcb:reset_switch.package]"
 			(at 0 0 90)
 			(layer "User.9")
@@
 			(fill no)
 			(layer "F.Fab")
-		)
-		(fp_text user "%R"
-			(at 0 0 90)
-			(layer "F.Fab")
-			(effects
-				(font
-					(size 1 1)
-					(thickness 0.15)
-				)
-			)
-		)
-		(fp_text user "${REFERENCE}"
-			(at 0 -5.07 90)
-			(layer "F.SilkS")
-			(effects
-				(font
-					(size 1 1)
-					(thickness 0.15)
-				)
-				(hide yes)
-			)
 		)
 		(pad "1" smd rect
@@
 			)
 		)
-		(property "Value" "10000Ω"
+		(property "Value" "10kΩ ±1%"
 			(at 0 4 180)
 			(layer "F.Fab")
@@
 			)
 		)
-		(property "resistance" "10000±1.0%Ω"
-			(at 0 0 0)
-			(layer "User.9")
-			(hide yes)
-			(effects
-				(font
-					(size 1 1)
-					(thickness 0.15)
-				)
-			)
-		)
-		(property "max_power" "0.062W"
+		(property "resistance" "10kΩ ±1%"
+			(at 0 0 0)
+			(layer "User.9")
+			(hide yes)
+			(effects
+				(font
+					(size 1 1)
+					(thickness 0.15)
+				)
+			)
+		)
+		(property "max_power" "62.5mW"
 			(at 0 0 0)
 			(layer "User.9")
@@
 			(layer "F.Fab")
 			(locked no)
-		)
-		(fp_text user "%R"
-			(at 0 0 180)
-			(layer "F.Fab")
-			(effects
-				(font
-					(size 1 1)
-					(thickness 0.15)
-				)
-			)
 		)
 		(pad "1" smd rect
@@
 			(layer "F.Fab")
 		)
-		(fp_text user "%R"
-			(at 0 0 0)
-			(layer "F.Fab")
-			(effects
-				(font
-					(size 1 1)
-					(thickness 0.15)
-				)
-			)
-		)
-		(fp_text user "${REFERENCE}"
-			(at 0 -12.89 0)
-			(layer "F.SilkS")
-			(effects
-				(font
-					(size 1 1)
-					(thickness 0.15)
-				)
-				(hide yes)
-			)
-		)
 		(pad "1" smd rect
 			(at -8.75 -8.89 0)
@@
 			)
 		)
-		(property "Value" "10000Ω"
+		(property "Value" "10kΩ ±1%"
 			(at 0 4 270)
 			(layer "F.Fab")
@@
 			)
 		)
-		(property "resistance" "10000±1.0%Ω"
-			(at 0 0 0)
-			(layer "User.9")
-			(hide yes)
-			(effects
-				(font
-					(size 1 1)
-					(thickness 0.15)
-				)
-			)
-		)
-		(property "max_power" "0.062W"
+		(property "resistance" "10kΩ ±1%"
+			(at 0 0 0)
+			(layer "User.9")
+			(hide yes)
+			(effects
+				(font
+					(size 1 1)
+					(thickness 0.15)
+				)
+			)
+		)
+		(property "max_power" "62.5mW"
 			(at 0 0 0)
 			(layer "User.9")
@@
 			(layer "F.Fab")
 			(locked no)
-		)
-		(fp_text user "%R"
-			(at 0 0 270)
-			(layer "F.Fab")
-			(effects
-				(font
-					(size 1 1)
-					(thickness 0.15)
-				)
-			)
 		)
 		(pad "1" smd rect
@@
 			)
 		)
-		(property "Value" "9.999F"
+		(property "Value" "10µF ±10%"
 			(at 0 4 90)
 			(layer "F.Fab")
@@
 			)
 		)
-		(property "capacitance" "9.999±10.0%F"
+		(property "capacitance" "10µF ±10%"
 			(at 0 0 0)
 			(layer "User.9")
@@
 			(layer "F.Fab")
 			(locked no)
-		)
-		(fp_text user "%R"
-			(at 0 0 90)
-			(layer "F.Fab")
-			(effects
-				(font
-					(size 1 1)
-					(thickness 0.15)
-				)
-			)
 		)
 		(pad "1" smd rect
@@
 			)
 		)
-		(property "atopile_subaddresses" "[layouts/default/default.kicad_pcb:boot_switch.package]"
+		(property "atopile_subaddresses" "[.ato/modules/atopile/buttons/layouts/VerticalButton/VerticalButton.kicad_pcb:package, layouts/default/default.kicad_pcb:boot_switch.package]"
 			(at 0 0 270)
 			(layer "User.9")
@@
 			(fill no)
 			(layer "F.Fab")
-		)
-		(fp_text user "%R"
-			(at 0 0 270)
-			(layer "F.Fab")
-			(effects
-				(font
-					(size 1 1)
-					(thickness 0.15)
-				)
-			)
-		)
-		(fp_text user "${REFERENCE}"
-			(at 0 -5.07 270)
-			(layer "F.SilkS")
-			(effects
-				(font
-					(size 1 1)
-					(thickness 0.15)
-				)
-				(hide yes)
-			)
 		)
 		(pad "1" smd rect
@@
 			)
 		)
-		(property "Value" "1e-06F"
+		(property "Value" "1µF ±10%"
 			(at 0 4 180)
 			(layer "F.Fab")
@@
 			)
 		)
-		(property "capacitance" "1e-06±10.0%F"
+		(property "capacitance" "1µF ±10%"
 			(at 0 0 0)
 			(layer "User.9")
@@
 			(layer "F.Fab")
 			(locked no)
-		)
-		(fp_text user "%R"
-			(at 0 0 180)
-			(layer "F.Fab")
-			(effects
-				(font
-					(size 1 1)
-					(thickness 0.15)
-				)
-			)
 		)
 		(pad "1" smd rect
@@
 			)
 		)
-		(property "Value" "1F"
+		(property "Value" "100nF ±10%"
 			(at 0 4 90)
 			(layer "F.Fab")
@@
 			)
 		)
-		(property "capacitance" "1±10.0%F"
+		(property "capacitance" "100nF ±10%"
 			(at 0 0 0)
 			(layer "User.9")
@@
 			(locked no)
 		)
-		(fp_text user "%R"
-			(at 0 0 90)
-			(layer "F.Fab")
-			(effects
-				(font
-					(size 1 1)
-					(thickness 0.15)
-				)
-			)
-		)
 		(pad "1" smd rect
